Commit message: transfer nao_robot

File: nao_description/urdf/naoV40_generated_urdf/naoGazebo.xacro (robot description, xacro)
@@ -75,5 +75,5 @@
             <robotSimType>gazebo_ros_control/DefaultRobotHWSim</robotSimType>
         </plugin>
-<!--        <plugin filename="libgazebo_ros_imu.so" name="gazebo_ros_imu_controller">
+        <plugin filename="libgazebo_ros_imu.so" name="gazebo_ros_imu_controller">
             <robotNamespace>/nao_dcm</robotNamespace>
             <topicName>imu_data</topicName>
@@ -89,5 +89,4 @@
             <alwaysOn>true</alwaysOn>
         </plugin>
--->
 <!--        <plugin name="gazebo_ros_imu_controller" filename="${imu_plugin}">
             <robotNamespace>/nao_dcm</robotNamespace>
@@ -424,235 +423,3 @@
         <turnGravityOff>true</turnGravityOff>
     </gazebo>
-<!--
-        RGB CAMERAS: Working
--->
- <gazebo reference="CameraTop_frame">
-    <sensor type="camera" name="CameraTop">
-        <update_rate>5.0</update_rate>
-        <camera name="camera_top">
-            <horizontal_fov>1.06290551</horizontal_fov>
-            <image>
-                <width>640</width>
-                <height>480</height>
-                <format>R8G8B8</format>
-            </image>
-            <clip>
-                <near>0.3</near>
-                <far>500</far>
-            </clip>
-            <noise>
-                <type>gaussian</type>
-                <mean>0.0</mean>
-                <stddev>0.007</stddev>
-            </noise>
-        </camera>
-        <plugin name="camera_controller" filename="libgazebo_ros_camera.so">
-            <robotNamespace>/nao_robot</robotNamespace>
-            <alwaysOn>true</alwaysOn>
-            <updateRate>5.0</updateRate>
-            <cameraName>camera/top</cameraName>
-            <imageTopicName>image_raw</imageTopicName>
-            <cameraInfoTopicName>camera_info</cameraInfoTopicName>
-            <frameName>CameraTop_frame</frameName>
-            <hackBaseline>0.07</hackBaseline>
-            <distortionK1>-0.0545211</distortionK1>
-            <distortionK2>0.06919734</distortionK2>
-            <distortionK3>-0.0241095</distortionK3>
-            <distortionT1>-0.0112245</distortionT1>
-            <distortionT2>0.0</distortionT2>
-        </plugin>
-    </sensor>
-</gazebo>
- <gazebo reference="CameraBottom_frame">
-    <sensor type="camera" name="CameraBottom">
-        <update_rate>5.0</update_rate>
-        <camera name="camera_bottom">
-            <horizontal_fov>1.06290551</horizontal_fov>
-            <image>
-                <width>640</width>
-                <height>480</height>
-                <format>R8G8B8</format>
-            </image>
-            <clip>
-                <near>0.3</near>
-                <far>500</far>
-            </clip>
-            <noise>
-                <type>gaussian</type>
-                <mean>0.0</mean>
-                <stddev>0.007</stddev>
-            </noise>
-        </camera>
-        <plugin name="camera_controller" filename="libgazebo_ros_camera.so">
-            <robotNamespace>/nao_robot</robotNamespace>
-            <alwaysOn>true</alwaysOn>
-            <updateRate>5.0</updateRate>
-            <cameraName>camera_bottom</cameraName>
-            <imageTopicName>image_raw</imageTopicName>
-            <cameraInfoTopicName>camera_info</cameraInfoTopicName>
-            <frameName>CameraBottom_frame</frameName>
-            <hackBaseline>0.07</hackBaseline>
-            <distortionK1>-0.0648764</distortionK1>
-            <distortionK2>0.06125202</distortionK2>
-            <distortionK3>0.00382815</distortionK3>
-            <distortionT1>-0.00551104</distortionT1>
-            <distortionT2>0.0</distortionT2>
-        </plugin>
-    </sensor>
-</gazebo>
-<!--
-        CameraDepth : not displayed at the right spot
-<gazebo reference="CameraDepth3_frame">
-    <sensor type="depth" name="openni_camera_camera2">
-        <always_on>1</always_on>
-        <visualize>true</visualize>
-        <camera>
-            <horizontal_fov>1.01229</horizontal_fov>
-            <image>
-                <width>320</width>
-                <height>240</height>
-                <format>R8G8B8</format>
-            </image>
-            <depth_camera>
-            </depth_camera>
-            <clip>
-                <near>0.1</near>
-                <far>100</far>
-            </clip>
-        </camera>
-        <plugin name="depth_cam_controller2" filename="libgazebo_ros_openni_kinect.so">
-            <baseline>0.2</baseline>
-            <alwaysOn>true</alwaysOn>
-            <updateRate>0.1</updateRate>
-            <cameraName>xtion2</cameraName>
-            <imageTopicName>/xtion2/ir/image_raw</imageTopicName>
-            <cameraInfoTopicName>/xtion2/ir/camera_info</cameraInfoTopicName>
-            <depthImageTopicName>/xtion2/depth/image_raw</depthImageTopicName>
-            <depthImageInfoTopicName>/xtion2/depth/camera_info</depthImageInfoTopicName>
-            <pointCloudTopicName>/xtion2/depth/points</pointCloudTopicName>
-            <frameName>CameraDepth2_frame</frameName>
-            <pointCloudCutoff>0.5</pointCloudCutoff>
-            <distortionK1>0.00000001</distortionK1>
-            <distortionK2>0.00000001</distortionK2>
-            <distortionK3>0.00000001</distortionK3>
-            <distortionT1>0.00000001</distortionT1>
-            <distortionT2>0.00000001</distortionT2>
-            <CxPrime>0</CxPrime>
-            <Cx>0</Cx>
-            <Cy>0</Cy>
-            <focalLength>0</focalLength>
-            <hackBaseline>0</hackBaseline>
-        </plugin>
-    </sensor>
-</gazebo>
--->
-<!--
-    BUMPERS
-libgazebo_ros_bumper.so bugged right now, waiting for new release
-<gazebo reference="LFootBumper_frame">
-  <sensor type="contact" name="LFootBumper">
-    <update_rate>10</update_rate>
-    <contact>
-      <collision>LFootBumper_frame_collision</collision>
-    </contact>
-    <plugin filename="libgazebo_ros_bumper.so" name="gazebo_nao_ros_bumper">
-      <alwaysOn>true</alwaysOn>
-      <bumperTopicName>lbumper</bumperTopicName>
-      <frameName>LFootBumper_frame</frameName>
-    </plugin>
-  </sensor>
-</gazebo>
--->
-<!--
-    Sonars : OK (except frame names)
--->
-<gazebo reference="LSonar_frame">
-  <sensor type="ray" name="LSonar">
-    <pose>0 0 0 0 0 0</pose>
-    <update_rate>20</update_rate>
-    <visualize>false</visualize>
-    <ray>
-      <scan>
-        <horizontal>
-          <samples>5</samples>
-          <resolution>1</resolution>
-          <min_angle>-0.2617993877991494</min_angle>
-          <max_angle>0.2617993877991494</max_angle>
-<!--
-          <min_angle>-0.10</min_angle>
-          <max_angle>0.10</max_angle>
--->
-        </horizontal>
-        <vertical>
-          <samples>5</samples>
-          <resolution>1</resolution>
-          <min_angle>-0.13</min_angle>
-          <max_angle>0.13</max_angle>
-<!--
-          <min_angle>-0.2617993877991494</min_angle>
-          <max_angle>0.2617993877991494</max_angle>
--->
-        </vertical>
-      </scan>
-      <range>
-        <min>0.025</min>
-        <max>2.55</max>
-        <resolution>1</resolution>
-      </range>
-    </ray>
-    <plugin filename="libgazebo_ros_range.so" name="gazebo_ros_range">
-      <robotNamespace>/nao_robot</robotNamespace>
-      <gaussianNoise>0.05</gaussianNoise>
-      <alwaysOn>true</alwaysOn>
-      <updateRate>20</updateRate>
-      <topicName>/sonar_left</topicName>
-      <frameName>LSonar_frame</frameName>
-      <minRange>0.025</minRange>
-      <maxRange>2.55</maxRange>
-      <fov>0.5235987755982988</fov>
-<!--      <fov>0.1</fov> -->
-      <radiation>ultrasound</radiation>
-    </plugin>
-  </sensor>
-</gazebo>
-<gazebo reference="RSonar_frame">
-  <sensor type="ray" name="RSonar">
-    <pose>0 0 0 0 0 0</pose>
-    <update_rate>20</update_rate>
-    <visualize>false</visualize>
-    <ray>
-      <scan>
-        <horizontal>
-          <samples>5</samples>
-          <resolution>1</resolution>
-          <min_angle>-0.2617993877991494</min_angle>
-          <max_angle>0.2617993877991494</max_angle>
-        </horizontal>
-        <vertical>
-          <samples>5</samples>
-          <resolution>1</resolution>
-          <min_angle>-0.13</min_angle>
-          <max_angle>0.13</max_angle>
-        </vertical>
-      </scan>
-      <range>
-        <min>0.025</min>
-        <max>2.55</max>
-        <resolution>1</resolution>
-      </range>
-    </ray>
-    <plugin filename="libgazebo_ros_range.so" name="gazebo_ros_range">
-      <robotNamespace>/nao_robot</robotNamespace>
-      <gaussianNoise>0.05</gaussianNoise>
-      <alwaysOn>true</alwaysOn>
-      <updateRate>20</updateRate>
-      <topicName>/sonar_right</topicName>
-      <frameName>RSonar_frame</frameName>
-      <minRange>0.025</minRange>
-      <maxRange>2.55</maxRange>
-      <fov>0.5235987755982988</fov>
-      <radiation>ultrasound</radiation>
-    </plugin>
-  </sensor>
-</gazebo>
 </robot>

File: nao_description/urdf/naoV40_generated_urdf/naosensors.xacro (robot description, xacro)
@@ -88,10 +88,4 @@
 		<origin rpy="0 0 0" xyz="0.0876 0.019 -0.035"/>
 	</joint>
-	<link name="LFootBumper_frame"/>
-	<joint name="LFootBumper_joint" type="fixed">
-		<parent link="l_ankle"/>
-		<child link="LFootBumper_frame"/>
-		<origin rpy="0 0 0" xyz="0.0876 0.0 -0.035"/>
-	</joint>
 	<link name="ChestButton_frame"/>
 	<joint name="ChestButton_joint" type="fixed">
@@ -148,51 +142,9 @@
 		<origin rpy="0 -1.186099535 0" xyz="0.0312 0 0.1014"/>
 	</joint>
-	<link name="CameraBottom_frame">
-    <inertial>
-        <mass value="0.05" />
-        <origin xyz="0 0 0" />
-        <inertia ixx="1e-9" ixy="0" ixz="0" iyy="1e-9" iyz="0" izz="1e-9" />
-    </inertial>
-    </link>
+	<link name="CameraBottom_frame"/>
 	<joint name="CameraBottom_joint" type="fixed">
 		<parent link="Head"/>
 		<child link="CameraBottom_frame"/>
 		<origin rpy="0 0.6929 0" xyz="0.05071 0 0.01774"/>
-	</joint>
-	<link name="CameraDepth_frame">
-    <inertial>
-        <mass value="0.05" />
-        <origin xyz="0 0 0" />
-        <inertia ixx="1e-9" ixy="0" ixz="0" iyy="1e-9" iyz="0" izz="1e-9" />
-    </inertial>
-    </link>
-	<joint name="CameraDepth_joint" type="fixed">
-		<parent link="Head"/>
-		<child link="CameraDepth_frame"/>
-		<origin rpy="1.05 3.14159265 1.57079632" xyz="-0.01 0.05 0.13"/>
-	</joint>
-	<link name="CameraDepth2_frame">
-    <inertial>
-        <mass value="0.05" />
-        <origin xyz="0 0 0" />
-        <inertia ixx="1e-9" ixy="0" ixz="0" iyy="1e-9" iyz="0" izz="1e-9" />
-    </inertial>
-    </link>
-	<joint name="CameraDepth2_joint" type="fixed">
-		<parent link="Head"/>
-		<child link="CameraDepth2_frame"/>
-		<origin rpy="0 -3.14159 1.5707" xyz="-0.01 0.05 0.13"/>
-	</joint>
-	<link name="CameraDepth3_frame">
-    <inertial>
-        <mass value="0.05" />
-        <origin xyz="0 0 0" />
-        <inertia ixx="1e-9" ixy="0" ixz="0" iyy="1e-9" iyz="0" izz="1e-9" />
-    </inertial>
-    </link>
-	<joint name="CameraDepth3_joint" type="fixed">
-		<parent link="Head"/>
-		<child link="CameraDepth3_frame"/>
-		<origin rpy="0 0 0" xyz="-0.01 0.05 0.13"/>
 	</joint>
 	<link name="LHandTouchRight_frame"/>
@@ -208,11 +160,5 @@
 		<origin rpy="0 0.04365 -0.39265" xyz="0.0507 -0.03785 0.06035"/>
 	</joint>
-	<link name="CameraTop_frame">
-    <inertial>
-        <mass value="0.05" />
-        <origin xyz="0 0 0" />
-        <inertia ixx="1e-9" ixy="0" ixz="0" iyy="1e-9" iyz="0" izz="1e-9" />
-    </inertial>
-    </link>
+	<link name="CameraTop_frame"/>
 	<joint name="CameraTop_joint" type="fixed">
 		<parent link="Head"/>

Commit message: Added camera and sonar sensor to gazebo urdf

File: nao_description/urdf/naoV40_generated_urdf/naoGazebo.xacro (robot description, xacro)
@@ -429,3 +429,235 @@
         <turnGravityOff>true</turnGravityOff>
     </gazebo>
+<!--
+        RGB CAMERAS: Working
+-->
+ <gazebo reference="CameraTop_frame">
+    <sensor type="camera" name="CameraTop">
+        <update_rate>5.0</update_rate>
+        <camera name="camera_top">
+            <horizontal_fov>1.06290551</horizontal_fov>
+            <image>
+                <width>640</width>
+                <height>480</height>
+                <format>R8G8B8</format>
+            </image>
+            <clip>
+                <near>0.3</near>
+                <far>500</far>
+            </clip>
+            <noise>
+                <type>gaussian</type>
+                <mean>0.0</mean>
+                <stddev>0.007</stddev>
+            </noise>
+        </camera>
+        <plugin name="camera_controller" filename="libgazebo_ros_camera.so">
+            <robotNamespace>/nao_robot</robotNamespace>
+            <alwaysOn>true</alwaysOn>
+            <updateRate>5.0</updateRate>
+            <cameraName>camera/top</cameraName>
+            <imageTopicName>image_raw</imageTopicName>
+            <cameraInfoTopicName>camera_info</cameraInfoTopicName>
+            <frameName>CameraTop_frame</frameName>
+            <hackBaseline>0.07</hackBaseline>
+            <distortionK1>-0.0545211</distortionK1>
+            <distortionK2>0.06919734</distortionK2>
+            <distortionK3>-0.0241095</distortionK3>
+            <distortionT1>-0.0112245</distortionT1>
+            <distortionT2>0.0</distortionT2>
+        </plugin>
+    </sensor>
+</gazebo>
+ <gazebo reference="CameraBottom_frame">
+    <sensor type="camera" name="CameraBottom">
+        <update_rate>5.0</update_rate>
+        <camera name="camera_bottom">
+            <horizontal_fov>1.06290551</horizontal_fov>
+            <image>
+                <width>640</width>
+                <height>480</height>
+                <format>R8G8B8</format>
+            </image>
+            <clip>
+                <near>0.3</near>
+                <far>500</far>
+            </clip>
+            <noise>
+                <type>gaussian</type>
+                <mean>0.0</mean>
+                <stddev>0.007</stddev>
+            </noise>
+        </camera>
+        <plugin name="camera_controller" filename="libgazebo_ros_camera.so">
+            <robotNamespace>/nao_robot</robotNamespace>
+            <alwaysOn>true</alwaysOn>
+            <updateRate>5.0</updateRate>
+            <cameraName>camera_bottom</cameraName>
+            <imageTopicName>image_raw</imageTopicName>
+            <cameraInfoTopicName>camera_info</cameraInfoTopicName>
+            <frameName>CameraBottom_frame</frameName>
+            <hackBaseline>0.07</hackBaseline>
+            <distortionK1>-0.0648764</distortionK1>
+            <distortionK2>0.06125202</distortionK2>
+            <distortionK3>0.00382815</distortionK3>
+            <distortionT1>-0.00551104</distortionT1>
+            <distortionT2>0.0</distortionT2>
+        </plugin>
+    </sensor>
+</gazebo>
+<!--
+        CameraDepth : not displayed at the right spot
+<gazebo reference="CameraDepth3_frame">
+    <sensor type="depth" name="openni_camera_camera2">
+        <always_on>1</always_on>
+        <visualize>true</visualize>
+        <camera>
+            <horizontal_fov>1.01229</horizontal_fov>
+            <image>
+                <width>320</width>
+                <height>240</height>
+                <format>R8G8B8</format>
+            </image>
+            <depth_camera>
+            </depth_camera>
+            <clip>
+                <near>0.1</near>
+                <far>100</far>
+            </clip>
+        </camera>
+        <plugin name="depth_cam_controller2" filename="libgazebo_ros_openni_kinect.so">
+            <baseline>0.2</baseline>
+            <alwaysOn>true</alwaysOn>
+            <updateRate>0.1</updateRate>
+            <cameraName>xtion2</cameraName>
+            <imageTopicName>/xtion2/ir/image_raw</imageTopicName>
+            <cameraInfoTopicName>/xtion2/ir/camera_info</cameraInfoTopicName>
+            <depthImageTopicName>/xtion2/depth/image_raw</depthImageTopicName>
+            <depthImageInfoTopicName>/xtion2/depth/camera_info</depthImageInfoTopicName>
+            <pointCloudTopicName>/xtion2/depth/points</pointCloudTopicName>
+            <frameName>CameraDepth2_frame</frameName>
+            <pointCloudCutoff>0.5</pointCloudCutoff>
+            <distortionK1>0.00000001</distortionK1>
+            <distortionK2>0.00000001</distortionK2>
+            <distortionK3>0.00000001</distortionK3>
+            <distortionT1>0.00000001</distortionT1>
+            <distortionT2>0.00000001</distortionT2>
+            <CxPrime>0</CxPrime>
+            <Cx>0</Cx>
+            <Cy>0</Cy>
+            <focalLength>0</focalLength>
+            <hackBaseline>0</hackBaseline>
+        </plugin>
+    </sensor>
+</gazebo>
+-->
+<!--
+    BUMPERS
+libgazebo_ros_bumper.so bugged right now, waiting for new release
+<gazebo reference="LFootBumper_frame">
+  <sensor type="contact" name="LFootBumper">
+    <update_rate>10</update_rate>
+    <contact>
+      <collision>LFootBumper_frame_collision</collision>
+    </contact>
+    <plugin filename="libgazebo_ros_bumper.so" name="gazebo_nao_ros_bumper">
+      <alwaysOn>true</alwaysOn>
+      <bumperTopicName>lbumper</bumperTopicName>
+      <frameName>LFootBumper_frame</frameName>
+    </plugin>
+  </sensor>
+</gazebo>
+-->
+<!--
+    Sonars : OK (except frame names)
+-->
+<gazebo reference="LSonar_frame">
+  <sensor type="ray" name="LSonar">
+    <pose>0 0 0 0 0 0</pose>
+    <update_rate>20</update_rate>
+    <visualize>false</visualize>
+    <ray>
+      <scan>
+        <horizontal>
+          <samples>5</samples>
+          <resolution>1</resolution>
+          <min_angle>-0.2617993877991494</min_angle>
+          <max_angle>0.2617993877991494</max_angle>
+<!--
+          <min_angle>-0.10</min_angle>
+          <max_angle>0.10</max_angle>
+-->
+        </horizontal>
+        <vertical>
+          <samples>5</samples>
+          <resolution>1</resolution>
+          <min_angle>-0.13</min_angle>
+          <max_angle>0.13</max_angle>
+<!--
+          <min_angle>-0.2617993877991494</min_angle>
+          <max_angle>0.2617993877991494</max_angle>
+-->
+        </vertical>
+      </scan>
+      <range>
+        <min>0.025</min>
+        <max>2.55</max>
+        <resolution>1</resolution>
+      </range>
+    </ray>
+    <plugin filename="libgazebo_ros_range.so" name="gazebo_ros_range">
+      <robotNamespace>/nao_robot</robotNamespace>
+      <gaussianNoise>0.05</gaussianNoise>
+      <alwaysOn>true</alwaysOn>
+      <updateRate>20</updateRate>
+      <topicName>/sonar_left</topicName>
+      <frameName>LSonar_frame</frameName>
+      <minRange>0.025</minRange>
+      <maxRange>2.55</maxRange>
+      <fov>0.5235987755982988</fov>
+<!--      <fov>0.1</fov> -->
+      <radiation>ultrasound</radiation>
+    </plugin>
+  </sensor>
+</gazebo>
+<gazebo reference="RSonar_frame">
+  <sensor type="ray" name="RSonar">
+    <pose>0 0 0 0 0 0</pose>
+    <update_rate>20</update_rate>
+    <visualize>false</visualize>
+    <ray>
+      <scan>
+        <horizontal>
+          <samples>5</samples>
+          <resolution>1</resolution>
+          <min_angle>-0.2617993877991494</min_angle>
+          <max_angle>0.2617993877991494</max_angle>
+        </horizontal>
+        <vertical>
+          <samples>5</samples>
+          <resolution>1</resolution>
+          <min_angle>-0.13</min_angle>
+          <max_angle>0.13</max_angle>
+        </vertical>
+      </scan>
+      <range>
+        <min>0.025</min>
+        <max>2.55</max>
+        <resolution>1</resolution>
+      </range>
+    </ray>
+    <plugin filename="libgazebo_ros_range.so" name="gazebo_ros_range">
+      <robotNamespace>/nao_robot</robotNamespace>
+      <gaussianNoise>0.05</gaussianNoise>
+      <alwaysOn>true</alwaysOn>
+      <updateRate>20</updateRate>
+      <topicName>/sonar_right</topicName>
+      <frameName>RSonar_frame</frameName>
+      <minRange>0.025</minRange>
+      <maxRange>2.55</maxRange>
+      <fov>0.5235987755982988</fov>
+      <radiation>ultrasound</radiation>
+    </plugin>
+  </sensor>
+</gazebo>
 </robot>
