Commit message: restore sensor in naoGazebo.xacro

File: nao_description/urdf/naoV40_generated_urdf/naoGazebo.xacro (robot description, xacro)
@@ -5,26 +5,26 @@
     <xacro:macro name="DisabledLinks" params="side side_small">
         <plugin name="${side}Finger11" filename="libroboticsgroup_gazebo_disable_link_plugin.so">
-            <link>${side}Finger11_link</link>
+            <link>${side}Finger11</link>
         </plugin>
         <plugin name="${side}Finger12" filename="libroboticsgroup_gazebo_disable_link_plugin.so">
-            <link>${side}Finger12_link</link>
+            <link>${side}Finger12</link>
         </plugin>
         <plugin name="${side}Finger13" filename="libroboticsgroup_gazebo_disable_link_plugin.so">
-            <link>${side}Finger13_link</link>
+            <link>${side}Finger13</link>
         </plugin>
         <plugin name="${side}Finger21" filename="libroboticsgroup_gazebo_disable_link_plugin.so">
-            <link>${side}Finger21_link</link>
+            <link>${side}Finger21</link>
         </plugin>
         <plugin name="${side}Finger22" filename="libroboticsgroup_gazebo_disable_link_plugin.so">
-            <link>${side}Finger22_link</link>
+            <link>${side}Finger22</link>
         </plugin>
         <plugin name="${side}Finger23" filename="libroboticsgroup_gazebo_disable_link_plugin.so">
-            <link>${side}Finger23_link</link>
+            <link>${side}Finger23</link>
         </plugin>
         <plugin name="${side}Thumb1" filename="libroboticsgroup_gazebo_disable_link_plugin.so">
-            <link>${side}Thumb1_link</link>
+            <link>${side}Thumb1</link>
         </plugin>
         <plugin name="${side}Thumb2" filename="libroboticsgroup_gazebo_disable_link_plugin.so">
-            <link>${side}Thumb2_link</link>
+            <link>${side}Thumb2</link>
         </plugin>
         <plugin name="${side_small}_gripper" filename="libroboticsgroup_gazebo_disable_link_plugin.so">
@@ -35,19 +35,19 @@
     <!-- Fingers -->
     <xacro:macro name="FingerMimics" params="side num">
-        <plugin name="mimic_${side}Finger${num}1" filename="libroboticsgroup_gazebo_mimic_joint_plugin.so">
+        <plugin name="mimic_${side}Finger${num}" filename="libroboticsgroup_gazebo_mimic_joint_plugin.so">
             <joint>${side}Hand</joint>
-            <mimicJoint>${side}Finger${num}1</mimicJoint>
+            <mimicJoint>${side}Finger${num}</mimicJoint>
             <multiplier>-${PI/4}</multiplier>
             <offset>${PI/4}</offset>
         </plugin>
-        <plugin name="mimic_${side}Finger${num}2" filename="libroboticsgroup_gazebo_mimic_joint_plugin.so">
+        <plugin name="mimic_${side}Finger${num}_1" filename="libroboticsgroup_gazebo_mimic_joint_plugin.so">
             <joint>${side}Hand</joint>
-            <mimicJoint>${side}Finger${num}2</mimicJoint>
+            <mimicJoint>${side}Finger${num}_1</mimicJoint>
             <multiplier>-${PI/4}</multiplier>
             <offset>${PI/4}</offset>
         </plugin>
-        <plugin name="mimic_${side}Finger${num}3" filename="libroboticsgroup_gazebo_mimic_joint_plugin.so">
+        <plugin name="mimic_${side}Finger${num}_2" filename="libroboticsgroup_gazebo_mimic_joint_plugin.so">
             <joint>${side}Hand</joint>
-            <mimicJoint>${side}Finger${num}3</mimicJoint>
+            <mimicJoint>${side}Finger${num}_2</mimicJoint>
             <multiplier>-${PI/4}</multiplier>
             <offset>${PI/4}</offset>
@@ -56,13 +56,13 @@
     <!-- Thumbs -->
     <xacro:macro name="ThumbMimics" params="side">
-        <plugin name="${side}Thumb1" filename="libroboticsgroup_gazebo_mimic_joint_plugin.so">
+        <plugin name="${side}Thumb1_joint" filename="libroboticsgroup_gazebo_mimic_joint_plugin.so">
             <joint>${side}Hand</joint>
-            <mimicJoint>${side}Thumb1</mimicJoint>
+            <mimicJoint>${side}Thumb1_joint</mimicJoint>
             <multiplier>-${PI/4}</multiplier>
             <offset>${PI/4}</offset>
         </plugin>
-        <plugin name="${side}Thumb2" filename="libroboticsgroup_gazebo_mimic_joint_plugin.so">
+        <plugin name="${side}Thumb1_2" filename="libroboticsgroup_gazebo_mimic_joint_plugin.so">
             <joint>${side}Hand</joint>
-            <mimicJoint>${side}Thumb2</mimicJoint>
+            <mimicJoint>${side}Thumb1_2</mimicJoint>
             <multiplier>-${PI/4}</multiplier>
             <offset>${PI/4}</offset>
@@ -75,4 +75,19 @@
             <robotSimType>gazebo_ros_control/DefaultRobotHWSim</robotSimType>
         </plugin>
+<!--        <plugin filename="libgazebo_ros_imu.so" name="gazebo_ros_imu_controller">
+            <robotNamespace>/nao_dcm</robotNamespace>
+            <topicName>imu_data</topicName>
+            <bodyName>imu</bodyName>
+            <frameId>ImuAccelerometer_frame</frameId>
+            <gaussianNoise>2.89e-08</gaussianNoise>
+            <accelGaussianNoise>2.89e-08 2.89e-08 2.89e-08</accelGaussianNoise>
+            <rateGaussianNoise>2.89e-08 2.89e-08 2.89e-08</rateGaussianNoise>
+            <headingGaussianNoise>2.89e-08 2.89e-08 2.89e-08</headingGaussianNoise>
+            <xyzOffsets>0 0 0</xyzOffsets>
+            <rpyOffsets>0 0 0</rpyOffsets>
+            <updateRate>30.0</updateRate>
+            <alwaysOn>true</alwaysOn>
+        </plugin>
+-->
 <!--        <plugin name="gazebo_ros_imu_controller" filename="${imu_plugin}">
             <robotNamespace>/nao_dcm</robotNamespace>
@@ -223,47 +238,47 @@
     </gazebo>
 -->
-    <gazebo reference="LFinger11_link">
-        <mu1>0.5</mu1>
-        <mu2>0.5</mu2>
-        <selfCollide>false</selfCollide>
-        <turnGravityOff>true</turnGravityOff>
-    </gazebo>
-    <gazebo reference="LFinger12_link">
-        <mu1>0.5</mu1>
-        <mu2>0.5</mu2>
-        <selfCollide>false</selfCollide>
-        <turnGravityOff>true</turnGravityOff>
-    </gazebo>
-    <gazebo reference="LFinger13_link">
-        <mu1>0.5</mu1>
-        <mu2>0.5</mu2>
-        <selfCollide>false</selfCollide>
-        <turnGravityOff>true</turnGravityOff>
-    </gazebo>
-    <gazebo reference="LFinger21_link">
-        <mu1>0.5</mu1>
-        <mu2>0.5</mu2>
-        <selfCollide>false</selfCollide>
-        <turnGravityOff>true</turnGravityOff>
-    </gazebo>
-    <gazebo reference="LFinger22_link">
-        <mu1>0.5</mu1>
-        <mu2>0.5</mu2>
-        <selfCollide>false</selfCollide>
-        <turnGravityOff>true</turnGravityOff>
-    </gazebo>
-    <gazebo reference="LFinger23_link">
-        <mu1>0.5</mu1>
-        <mu2>0.5</mu2>
-        <selfCollide>false</selfCollide>
-        <turnGravityOff>true</turnGravityOff>
-    </gazebo>
-    <gazebo reference="LThumb1_link">
-        <mu1>0.5</mu1>
-        <mu2>0.5</mu2>
-        <selfCollide>false</selfCollide>
-        <turnGravityOff>true</turnGravityOff>
-    </gazebo>
-    <gazebo reference="LThumb2_link">
+    <gazebo reference="LFinger11">
+        <mu1>0.5</mu1>
+        <mu2>0.5</mu2>
+        <selfCollide>false</selfCollide>
+        <turnGravityOff>true</turnGravityOff>
+    </gazebo>
+    <gazebo reference="LFinger12">
+        <mu1>0.5</mu1>
+        <mu2>0.5</mu2>
+        <selfCollide>false</selfCollide>
+        <turnGravityOff>true</turnGravityOff>
+    </gazebo>
+    <gazebo reference="LFinger13">
+        <mu1>0.5</mu1>
+        <mu2>0.5</mu2>
+        <selfCollide>false</selfCollide>
+        <turnGravityOff>true</turnGravityOff>
+    </gazebo>
+    <gazebo reference="LFinger21">
+        <mu1>0.5</mu1>
+        <mu2>0.5</mu2>
+        <selfCollide>false</selfCollide>
+        <turnGravityOff>true</turnGravityOff>
+    </gazebo>
+    <gazebo reference="LFinger22">
+        <mu1>0.5</mu1>
+        <mu2>0.5</mu2>
+        <selfCollide>false</selfCollide>
+        <turnGravityOff>true</turnGravityOff>
+    </gazebo>
+    <gazebo reference="LFinger23">
+        <mu1>0.5</mu1>
+        <mu2>0.5</mu2>
+        <selfCollide>false</selfCollide>
+        <turnGravityOff>true</turnGravityOff>
+    </gazebo>
+    <gazebo reference="LThumb1">
+        <mu1>0.5</mu1>
+        <mu2>0.5</mu2>
+        <selfCollide>false</selfCollide>
+        <turnGravityOff>true</turnGravityOff>
+    </gazebo>
+    <gazebo reference="LThumb2">
         <mu1>0.5</mu1>
         <mu2>0.5</mu2>
@@ -295,11 +310,18 @@
         <turnGravityOff>false</turnGravityOff>
     </gazebo>
-    <gazebo reference="LAnklePitch">
-        <mu1>0.5</mu1>
-        <mu2>0.5</mu2>
-        <selfCollide>false</selfCollide>
-        <turnGravityOff>false</turnGravityOff>
-    </gazebo>
     <gazebo reference="l_ankle">
+        <mu1>0.5</mu1>
+        <mu2>0.5</mu2>
+        <selfCollide>false</selfCollide>
+        <turnGravityOff>false</turnGravityOff>
+    </gazebo>
+<!--    <gazebo reference="LFeet">
+        <mu1>0.5</mu1>
+        <mu2>0.5</mu2>
+        <selfCollide>false</selfCollide>
+        <turnGravityOff>false</turnGravityOff>
+    </gazebo> -->
+<!--
+    <gazebo reference="l_sole">
         <mu1>0.5</mu1>
         <mu2>0.5</mu2>
@@ -310,12 +332,57 @@
         <minDepth>0.003</minDepth>
     </gazebo>
-<!--
-    <gazebo reference="l_ankle">
-        <mu1>0.5</mu1>
-        <mu2>0.5</mu2>
-        <selfCollide>false</selfCollide>
-        <turnGravityOff>false</turnGravityOff>
-    </gazebo>
-    <gazebo reference="l_sole">
+-->
+ <gazebo reference="LAnklePitch">
+    <mu1>0.5</mu1>
+    <mu2>0.5</mu2>
+    <selfCollide>false</selfCollide>
+    <turnGravityOff>false</turnGravityOff>
+  </gazebo>
+  <gazebo reference="l_ankle">
+    <mu1>0.5</mu1>
+    <mu2>0.5</mu2>
+    <selfCollide>false</selfCollide>
+    <turnGravityOff>false</turnGravityOff>
+    <fdir1>1 0 0</fdir1>
+    <maxVel>0.1</maxVel>
+    <minDepth>0.003</minDepth>
+  </gazebo>
+    <gazebo reference="RPelvis">
+        <mu1>0.5</mu1>
+        <mu2>0.5</mu2>
+        <selfCollide>false</selfCollide>
+        <turnGravityOff>false</turnGravityOff>
+    </gazebo>
+    <gazebo reference="RHip">
+        <mu1>0.5</mu1>
+        <mu2>0.5</mu2>
+        <selfCollide>false</selfCollide>
+        <turnGravityOff>false</turnGravityOff>
+    </gazebo>
+    <gazebo reference="RThigh">
+        <mu1>0.5</mu1>
+        <mu2>0.5</mu2>
+        <selfCollide>false</selfCollide>
+        <turnGravityOff>false</turnGravityOff>
+    </gazebo>
+    <gazebo reference="RTibia">
+        <mu1>0.5</mu1>
+        <mu2>0.5</mu2>
+        <selfCollide>false</selfCollide>
+        <turnGravityOff>false</turnGravityOff>
+    </gazebo>
+<!--    <gazebo reference="r_ankle">
+        <mu1>0.5</mu1>
+        <mu2>0.5</mu2>
+        <selfCollide>false</selfCollide>
+        <turnGravityOff>false</turnGravityOff>
+    </gazebo> -->
+<!--    <gazebo reference="RFeet">
+        <mu1>0.5</mu1>
+        <mu2>0.5</mu2>
+        <selfCollide>false</selfCollide>
+        <turnGravityOff>false</turnGravityOff>
+    </gazebo> -->
+<!--    <gazebo reference="r_sole">
         <mu1>0.5</mu1>
         <mu2>0.5</mu2>
@@ -327,105 +394,298 @@
     </gazebo>
 -->
-    <gazebo reference="RPelvis">
-        <mu1>0.5</mu1>
-        <mu2>0.5</mu2>
-        <selfCollide>false</selfCollide>
-        <turnGravityOff>false</turnGravityOff>
-    </gazebo>
-    <gazebo reference="RHip">
-        <mu1>0.5</mu1>
-        <mu2>0.5</mu2>
-        <selfCollide>false</selfCollide>
-        <turnGravityOff>false</turnGravityOff>
-    </gazebo>
-    <gazebo reference="RThigh">
-        <mu1>0.5</mu1>
-        <mu2>0.5</mu2>
-        <selfCollide>false</selfCollide>
-        <turnGravityOff>false</turnGravityOff>
-    </gazebo>
-    <gazebo reference="RTibia">
-        <mu1>0.5</mu1>
-        <mu2>0.5</mu2>
-        <selfCollide>false</selfCollide>
-        <turnGravityOff>false</turnGravityOff>
-    </gazebo>
-<!--    <gazebo reference="r_ankle">
-        <mu1>0.5</mu1>
-        <mu2>0.5</mu2>
-        <selfCollide>false</selfCollide>
-        <turnGravityOff>false</turnGravityOff>
-    </gazebo> -->
-<!--    <gazebo reference="r_sole">
-        <mu1>0.5</mu1>
-        <mu2>0.5</mu2>
-        <selfCollide>false</selfCollide>
-        <turnGravityOff>false</turnGravityOff>
-        <fdir1>1 0 0</fdir1>
-        <maxVel>0.1</maxVel>
-        <minDepth>0.003</minDepth>
-    </gazebo> -->
-    <gazebo reference="RAnklePitch">
-        <mu1>0.5</mu1>
-        <mu2>0.5</mu2>
-        <selfCollide>false</selfCollide>
-        <turnGravityOff>false</turnGravityOff>
-    </gazebo>
-    <gazebo reference="r_ankle">
-        <mu1>0.5</mu1>
-        <mu2>0.5</mu2>
-        <selfCollide>false</selfCollide>
-        <turnGravityOff>false</turnGravityOff>
-        <fdir1>1 0 0</fdir1>
-        <maxVel>0.1</maxVel>
-        <minDepth>0.003</minDepth>
-    </gazebo>
-    <gazebo reference="RFinger11_link">
-        <mu1>0.5</mu1>
-        <mu2>0.5</mu2>
-        <selfCollide>false</selfCollide>
-        <turnGravityOff>true</turnGravityOff>
-    </gazebo>
-    <gazebo reference="RFinger12_link">
-        <mu1>0.5</mu1>
-        <mu2>0.5</mu2>
-        <selfCollide>false</selfCollide>
-        <turnGravityOff>true</turnGravityOff>
-    </gazebo>
-    <gazebo reference="RFinger13_link">
-        <mu1>0.5</mu1>
-        <mu2>0.5</mu2>
-        <selfCollide>false</selfCollide>
-        <turnGravityOff>true</turnGravityOff>
-    </gazebo>
-    <gazebo reference="RFinger21_link">
-        <mu1>0.5</mu1>
-        <mu2>0.5</mu2>
-        <selfCollide>false</selfCollide>
-        <turnGravityOff>true</turnGravityOff>
-    </gazebo>
-    <gazebo reference="RFinger22_link">
-        <mu1>0.5</mu1>
-        <mu2>0.5</mu2>
-        <selfCollide>false</selfCollide>
-        <turnGravityOff>true</turnGravityOff>
-    </gazebo>
-    <gazebo reference="RFinger23_link">
-        <mu1>0.5</mu1>
-        <mu2>0.5</mu2>
-        <selfCollide>false</selfCollide>
-        <turnGravityOff>true</turnGravityOff>
-    </gazebo>
-    <gazebo reference="RThumb1_link">
-        <mu1>0.5</mu1>
-        <mu2>0.5</mu2>
-        <selfCollide>false</selfCollide>
-        <turnGravityOff>true</turnGravityOff>
-    </gazebo>
-    <gazebo reference="RThumb2_link">
-        <mu1>0.5</mu1>
-        <mu2>0.5</mu2>
-        <selfCollide>false</selfCollide>
-        <turnGravityOff>true</turnGravityOff>
-    </gazebo>
+ <gazebo reference="RAnklePitch">
+    <mu1>0.5</mu1>
+    <mu2>0.5</mu2>
+    <selfCollide>false</selfCollide>
+    <turnGravityOff>false</turnGravityOff>
+  </gazebo>
+  <gazebo reference="r_ankle">
+    <mu1>0.5</mu1>
+    <mu2>0.5</mu2>
+    <selfCollide>false</selfCollide>
+    <turnGravityOff>false</turnGravityOff>
+    <fdir1>1 0 0</fdir1>
+    <maxVel>0.1</maxVel>
+    <minDepth>0.003</minDepth>
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
File: nao_description/urdf/naoV40_generated_urdf/nao_sensors.xacro (robot description, xacro)
@@ -74,8 +74,8 @@
 		<axis xyz="0 0 0"/>
 	</joint>
-	<link name="LSonar_frame"/>
+	<link name="RSonar_frame"/>
 	<joint name="Sonar/Right_sensor_fixedjoint" type="fixed">
 		<parent link="torso"/>
-		<child link="LSonar_frame"/>
+		<child link="RSonar_frame"/>
 		<origin rpy="0.00478508 0.0436497 -0.392441" xyz="0.00558253 -0.0192068 0.0623853"/>
 		<axis xyz="0 0 0"/>
@@ -151,8 +151,8 @@
 		<axis xyz="0 0 0"/>
 	</joint>
-	<link name="RSonar_frame"/>
+	<link name="LSonar_frame"/>
 	<joint name="Sonar/Left_sensor_fixedjoint" type="fixed">
 		<parent link="torso"/>
-		<child link="RSonar_frame"/>
+		<child link="LSonar_frame"/>
 		<origin rpy="-0.00478508 0.0436497 0.392441" xyz="0.00558253 0.0192068 0.0623853"/>
 		<axis xyz="0 0 0"/>
