Commit message: update to the latest version of the generation script

File: nao_description/urdf/naoV32_generated_urdf/nao_arms.xacro (robot description, xacro)
@@ -85,10 +85,5 @@
 		<limit effort="0.292" lower="0" upper="1.0" velocity="3.71"/>
 	</joint>
-	<link name="l_gripper">
-		<inertial>
-			<mass value="2e-06"/>
-			<inertia ixx="1.1e-09" ixy="0" ixz="0" iyy="1.1e-09" iyz="0" izz="1.1e-09"/>
-		</inertial>
-	</link>
+	<link name="l_gripper"/>
 	<joint name="RShoulderPitch" type="revolute">
 		<parent link="torso"/>
@@ -172,9 +167,4 @@
 		<limit effort="0.292" lower="0" upper="1.0" velocity="3.71"/>
 	</joint>
-	<link name="r_gripper">
-		<inertial>
-			<mass value="2e-06"/>
-			<inertia ixx="1.1e-09" ixy="0" ixz="0" iyy="1.1e-09" iyz="0" izz="1.1e-09"/>
-		</inertial>
-	</link>
+	<link name="r_gripper"/>
 </robot>

File: nao_description/urdf/naoV32_generated_urdf/nao_fingers.xacro (robot description, xacro)
@@ -5,8 +5,4 @@
 <robot name="naoH25V32" xmlns:xacro="http://www.ros.org/wiki/xacro">
 	<link name="RFinger13_link">
-		<inertial>
-			<mass value="2e-06"/>
-			<inertia ixx="1.1e-09" ixy="0" ixz="0" iyy="1.1e-09" iyz="0" izz="1.1e-09"/>
-		</inertial>
 		<xacro:insert_visu_RFinger13_link/>
 	</link>
@@ -19,8 +15,4 @@
 	</joint>
 	<link name="RFinger12_link">
-		<inertial>
-			<mass value="2e-06"/>
-			<inertia ixx="1.1e-09" ixy="0" ixz="0" iyy="1.1e-09" iyz="0" izz="1.1e-09"/>
-		</inertial>
 		<xacro:insert_visu_RFinger12_link/>
 	</link>
@@ -33,8 +25,4 @@
 	</joint>
 	<link name="LFinger21_link">
-		<inertial>
-			<mass value="2e-06"/>
-			<inertia ixx="1.1e-09" ixy="0" ixz="0" iyy="1.1e-09" iyz="0" izz="1.1e-09"/>
-		</inertial>
 		<xacro:insert_visu_LFinger21_link/>
 	</link>
@@ -47,8 +35,4 @@
 	</joint>
 	<link name="LFinger13_link">
-		<inertial>
-			<mass value="2e-06"/>
-			<inertia ixx="1.1e-09" ixy="0" ixz="0" iyy="1.1e-09" iyz="0" izz="1.1e-09"/>
-		</inertial>
 		<xacro:insert_visu_LFinger13_link/>
 	</link>
@@ -61,8 +45,4 @@
 	</joint>
 	<link name="LFinger11_link">
-		<inertial>
-			<mass value="2e-06"/>
-			<inertia ixx="1.1e-09" ixy="0" ixz="0" iyy="1.1e-09" iyz="0" izz="1.1e-09"/>
-		</inertial>
 		<xacro:insert_visu_LFinger11_link/>
 	</link>
@@ -75,8 +55,4 @@
 	</joint>
 	<link name="RFinger22_link">
-		<inertial>
-			<mass value="2e-06"/>
-			<inertia ixx="1.1e-09" ixy="0" ixz="0" iyy="1.1e-09" iyz="0" izz="1.1e-09"/>
-		</inertial>
 		<xacro:insert_visu_RFinger22_link/>
 	</link>
@@ -89,8 +65,4 @@
 	</joint>
 	<link name="LFinger22_link">
-		<inertial>
-			<mass value="2e-06"/>
-			<inertia ixx="1.1e-09" ixy="0" ixz="0" iyy="1.1e-09" iyz="0" izz="1.1e-09"/>
-		</inertial>
 		<xacro:insert_visu_LFinger22_link/>
 	</link>
@@ -103,8 +75,4 @@
 	</joint>
 	<link name="RFinger21_link">
-		<inertial>
-			<mass value="2e-06"/>
-			<inertia ixx="1.1e-09" ixy="0" ixz="0" iyy="1.1e-09" iyz="0" izz="1.1e-09"/>
-		</inertial>
 		<xacro:insert_visu_RFinger21_link/>
 	</link>
@@ -117,8 +85,4 @@
 	</joint>
 	<link name="LFinger12_link">
-		<inertial>
-			<mass value="2e-06"/>
-			<inertia ixx="1.1e-09" ixy="0" ixz="0" iyy="1.1e-09" iyz="0" izz="1.1e-09"/>
-		</inertial>
 		<xacro:insert_visu_LFinger12_link/>
 	</link>
@@ -131,8 +95,4 @@
 	</joint>
 	<link name="RFinger23_link">
-		<inertial>
-			<mass value="2e-06"/>
-			<inertia ixx="1.1e-09" ixy="0" ixz="0" iyy="1.1e-09" iyz="0" izz="1.1e-09"/>
-		</inertial>
 		<xacro:insert_visu_RFinger23_link/>
 	</link>
@@ -145,8 +105,4 @@
 	</joint>
 	<link name="RFinger11_link">
-		<inertial>
-			<mass value="2e-06"/>
-			<inertia ixx="1.1e-09" ixy="0" ixz="0" iyy="1.1e-09" iyz="0" izz="1.1e-09"/>
-		</inertial>
 		<xacro:insert_visu_RFinger11_link/>
 	</link>
@@ -159,8 +115,4 @@
 	</joint>
 	<link name="LFinger23_link">
-		<inertial>
-			<mass value="2e-06"/>
-			<inertia ixx="1.1e-09" ixy="0" ixz="0" iyy="1.1e-09" iyz="0" izz="1.1e-09"/>
-		</inertial>
 		<xacro:insert_visu_LFinger23_link/>
 	</link>
@@ -173,8 +125,4 @@
 	</joint>
 	<link name="LThumb1_link">
-		<inertial>
-			<mass value="2e-06"/>
-			<inertia ixx="1.1e-09" ixy="0" ixz="0" iyy="1.1e-09" iyz="0" izz="1.1e-09"/>
-		</inertial>
 		<xacro:insert_visu_LThumb1_link/>
 	</link>
@@ -187,8 +135,4 @@
 	</joint>
 	<link name="RThumb1_link">
-		<inertial>
-			<mass value="2e-06"/>
-			<inertia ixx="1.1e-09" ixy="0" ixz="0" iyy="1.1e-09" iyz="0" izz="1.1e-09"/>
-		</inertial>
 		<xacro:insert_visu_RThumb1_link/>
 	</link>
@@ -201,8 +145,4 @@
 	</joint>
 	<link name="RThumb2_link">
-		<inertial>
-			<mass value="2e-06"/>
-			<inertia ixx="1.1e-09" ixy="0" ixz="0" iyy="1.1e-09" iyz="0" izz="1.1e-09"/>
-		</inertial>
 		<xacro:insert_visu_RThumb2_link/>
 	</link>
@@ -215,8 +155,4 @@
 	</joint>
 	<link name="LThumb2_link">
-		<inertial>
-			<mass value="2e-06"/>
-			<inertia ixx="1.1e-09" ixy="0" ixz="0" iyy="1.1e-09" iyz="0" izz="1.1e-09"/>
-		</inertial>
 		<xacro:insert_visu_LThumb2_link/>
 	</link>

File: nao_description/urdf/naoV32_generated_urdf/nao_sensors.xacro (robot description, xacro)
@@ -18,4 +18,10 @@
 		<axis xyz="0 0 0"/>
 	</joint>
+	<link name="CameraBottom_optical_frame"/>
+	<joint name="CameraBottom_optical_frame_joint" type="fixed">
+		<parent link="CameraBottom_frame"/>
+		<child link="CameraBottom_optical_frame"/>
+		<origin rpy="-1.57079632679 0 -1.57079632679" xyz="0 0 0"/>
+	</joint>
 	<link name="RFsrRR_frame"/>
 	<joint name="RFoot/FSR/RearRight_sensor_fixedjoint" type="fixed">
@@ -81,4 +87,73 @@
 		<axis xyz="0 0 0"/>
 	</joint>
+	<link name="RSonar_frame"/>
+	<joint name="Sonar/Right_sensor_fixedjoint" type="fixed">
+		<parent link="torso"/>
+		<child link="RSonar_frame"/>
+		<origin rpy="0.00478508 0.0436497 -0.392441" xyz="0.00558253 -0.0192068 0.0623853"/>
+		<axis xyz="0 0 0"/>
+	</joint>
+	<link name="RFsrFL_frame"/>
+	<joint name="RFoot/FSR/FrontLeft_sensor_fixedjoint" type="fixed">
+		<parent link="r_ankle"/>
+		<child link="RFsrFL_frame"/>
+		<origin rpy="0 0 0" xyz="0.07025 0.0231 -0.04511"/>
+		<axis xyz="0 0 0"/>
+	</joint>
+	<link name="MicroSurroundRight_frame"/>
+	<joint name="MicroRight_sensor_fixedjoint" type="fixed">
+		<parent link="Head"/>
+		<child link="MicroSurroundRight_frame"/>
+		<origin rpy="0 0 0" xyz="-0.0195 -0.0606 0.0331"/>
+		<axis xyz="0 0 0"/>
+	</joint>
+	<link name="LSonar_frame"/>
+	<joint name="Sonar/Left_sensor_fixedjoint" type="fixed">
+		<parent link="torso"/>
+		<child link="LSonar_frame"/>
+		<origin rpy="-0.00478508 0.0436497 0.392441" xyz="0.00558253 0.0192068 0.0623853"/>
+		<axis xyz="0 0 0"/>
+	</joint>
+	<link name="LFsrFL_frame"/>
+	<joint name="LFoot/FSR/FrontLeft_sensor_fixedjoint" type="fixed">
+		<parent link="l_ankle"/>
+		<child link="LFsrFL_frame"/>
+		<origin rpy="0 0 0" xyz="0.07025 0.0299 -0.04511"/>
+		<axis xyz="0 0 0"/>
+	</joint>
+	<link name="LFsrRL_frame"/>
+	<joint name="LFoot/FSR/RearLeft_sensor_fixedjoint" type="fixed">
+		<parent link="l_ankle"/>
+		<child link="LFsrRL_frame"/>
+		<origin rpy="0 0 0" xyz="-0.03025 0.0299 -0.04511"/>
+		<axis xyz="0 0 0"/>
+	</joint>
+	<link name="CameraBottom_frame"/>
+	<joint name="CameraBottom_sensor_fixedjoint" type="fixed">
+		<parent link="Head"/>
+		<child link="CameraBottom_frame"/>
+		<origin rpy="0 0.6981 0" xyz="0.0488 0 0.02381"/>
+		<axis xyz="0 0 0"/>
+	</joint>
+	<link name="CameraTop_frame"/>
+	<joint name="CameraTop_sensor_fixedjoint" type="fixed">
+		<parent link="Head"/>
+		<child link="CameraTop_frame"/>
+		<origin rpy="0 0 0" xyz="0.0539 0 0.0679"/>
+		<axis xyz="0 0 0"/>
+	</joint>
+	<link name="CameraTop_optical_frame"/>
+	<joint name="CameraTop_optical_frame_joint" type="fixed">
+		<parent link="CameraTop_frame"/>
+		<child link="CameraTop_optical_frame"/>
+		<origin rpy="-1.57079632679 0 -1.57079632679" xyz="0 0 0"/>
+	</joint>
+	<link name="LInfraRed_frame"/>
+	<joint name="InfraredL_sensor_fixedjoint" type="fixed">
+		<parent link="Head"/>
+		<child link="LInfraRed_frame"/>
+		<origin rpy="0 0 0" xyz="0.0441 0.0257 0.0466"/>
+		<axis xyz="0 0 0"/>
+	</joint>
 	<link name="ImuTorsoGyrometer_frame"/>
 	<joint name="Gyrometer_sensor_fixedjoint" type="fixed">
@@ -88,67 +163,4 @@
 		<axis xyz="0 0 0"/>
 	</joint>
-	<link name="RFsrFL_frame"/>
-	<joint name="RFoot/FSR/FrontLeft_sensor_fixedjoint" type="fixed">
-		<parent link="r_ankle"/>
-		<child link="RFsrFL_frame"/>
-		<origin rpy="0 0 0" xyz="0.07025 0.0231 -0.04511"/>
-		<axis xyz="0 0 0"/>
-	</joint>
-	<link name="MicroSurroundRight_frame"/>
-	<joint name="MicroRight_sensor_fixedjoint" type="fixed">
-		<parent link="Head"/>
-		<child link="MicroSurroundRight_frame"/>
-		<origin rpy="0 0 0" xyz="-0.0195 -0.0606 0.0331"/>
-		<axis xyz="0 0 0"/>
-	</joint>
-	<link name="LSonar_frame"/>
-	<joint name="Sonar/Right_sensor_fixedjoint" type="fixed">
-		<parent link="torso"/>
-		<child link="LSonar_frame"/>
-		<origin rpy="0.00478508 0.0436497 -0.392441" xyz="0.00558253 -0.0192068 0.0623853"/>
-		<axis xyz="0 0 0"/>
-	</joint>
-	<link name="LFsrFL_frame"/>
-	<joint name="LFoot/FSR/FrontLeft_sensor_fixedjoint" type="fixed">
-		<parent link="l_ankle"/>
-		<child link="LFsrFL_frame"/>
-		<origin rpy="0 0 0" xyz="0.07025 0.0299 -0.04511"/>
-		<axis xyz="0 0 0"/>
-	</joint>
-	<link name="LFsrRL_frame"/>
-	<joint name="LFoot/FSR/RearLeft_sensor_fixedjoint" type="fixed">
-		<parent link="l_ankle"/>
-		<child link="LFsrRL_frame"/>
-		<origin rpy="0 0 0" xyz="-0.03025 0.0299 -0.04511"/>
-		<axis xyz="0 0 0"/>
-	</joint>
-	<link name="CameraBottom_frame"/>
-	<joint name="CameraBottom_sensor_fixedjoint" type="fixed">
-		<parent link="Head"/>
-		<child link="CameraBottom_frame"/>
-		<origin rpy="0 0.6981 0" xyz="0.0488 0 0.02381"/>
-		<axis xyz="0 0 0"/>
-	</joint>
-	<link name="CameraTop_frame"/>
-	<joint name="CameraTop_sensor_fixedjoint" type="fixed">
-		<parent link="Head"/>
-		<child link="CameraTop_frame"/>
-		<origin rpy="0 0 0" xyz="0.0539 0 0.0679"/>
-		<axis xyz="0 0 0"/>
-	</joint>
-	<link name="LInfraRed_frame"/>
-	<joint name="InfraredL_sensor_fixedjoint" type="fixed">
-		<parent link="Head"/>
-		<child link="LInfraRed_frame"/>
-		<origin rpy="0 0 0" xyz="0.0441 0.0257 0.0466"/>
-		<axis xyz="0 0 0"/>
-	</joint>
-	<link name="RSonar_frame"/>
-	<joint name="Sonar/Left_sensor_fixedjoint" type="fixed">
-		<parent link="torso"/>
-		<child link="RSonar_frame"/>
-		<origin rpy="-0.00478508 0.0436497 0.392441" xyz="0.00558253 0.0192068 0.0623853"/>
-		<axis xyz="0 0 0"/>
-	</joint>
 	<link name="MicroFrontCenter_frame"/>
 	<joint name="MicroFront_sensor_fixedjoint" type="fixed">

File: nao_description/urdf/naoV33_generated_urdf/nao_arms.xacro (robot description, xacro)
@@ -85,10 +85,5 @@
 		<limit effort="0.292" lower="0" upper="1.0" velocity="8.33"/>
 	</joint>
-	<link name="l_gripper">
-		<inertial>
-			<mass value="2e-06"/>
-			<inertia ixx="1.1e-09" ixy="0" ixz="0" iyy="1.1e-09" iyz="0" izz="1.1e-09"/>
-		</inertial>
-	</link>
+	<link name="l_gripper"/>
 	<joint name="RShoulderPitch" type="revolute">
 		<parent link="torso"/>
@@ -172,9 +167,4 @@
 		<limit effort="0.292" lower="0" upper="1.0" velocity="8.33"/>
 	</joint>
-	<link name="r_gripper">
-		<inertial>
-			<mass value="2e-06"/>
-			<inertia ixx="1.1e-09" ixy="0" ixz="0" iyy="1.1e-09" iyz="0" izz="1.1e-09"/>
-		</inertial>
-	</link>
+	<link name="r_gripper"/>
 </robot>

File: nao_description/urdf/naoV33_generated_urdf/nao_fingers.xacro (robot description, xacro)
@@ -5,8 +5,4 @@
 <robot name="naoH25V33" xmlns:xacro="http://www.ros.org/wiki/xacro">
 	<link name="RFinger13_link">
-		<inertial>
-			<mass value="2e-06"/>
-			<inertia ixx="1.1e-09" ixy="0" ixz="0" iyy="1.1e-09" iyz="0" izz="1.1e-09"/>
-		</inertial>
 		<xacro:insert_visu_RFinger13_link/>
 	</link>
@@ -19,8 +15,4 @@
 	</joint>
 	<link name="RFinger12_link">
-		<inertial>
-			<mass value="2e-06"/>
-			<inertia ixx="1.1e-09" ixy="0" ixz="0" iyy="1.1e-09" iyz="0" izz="1.1e-09"/>
-		</inertial>
 		<xacro:insert_visu_RFinger12_link/>
 	</link>
@@ -33,8 +25,4 @@
 	</joint>
 	<link name="LFinger21_link">
-		<inertial>
-			<mass value="2e-06"/>
-			<inertia ixx="1.1e-09" ixy="0" ixz="0" iyy="1.1e-09" iyz="0" izz="1.1e-09"/>
-		</inertial>
 		<xacro:insert_visu_LFinger21_link/>
 	</link>
@@ -47,8 +35,4 @@
 	</joint>
 	<link name="LFinger13_link">
-		<inertial>
-			<mass value="2e-06"/>
-			<inertia ixx="1.1e-09" ixy="0" ixz="0" iyy="1.1e-09" iyz="0" izz="1.1e-09"/>
-		</inertial>
 		<xacro:insert_visu_LFinger13_link/>
 	</link>
@@ -61,8 +45,4 @@
 	</joint>
 	<link name="LFinger11_link">
-		<inertial>
-			<mass value="2e-06"/>
-			<inertia ixx="1.1e-09" ixy="0" ixz="0" iyy="1.1e-09" iyz="0" izz="1.1e-09"/>
-		</inertial>
 		<xacro:insert_visu_LFinger11_link/>
 	</link>
@@ -75,8 +55,4 @@
 	</joint>
 	<link name="RFinger22_link">
-		<inertial>
-			<mass value="2e-06"/>
-			<inertia ixx="1.1e-09" ixy="0" ixz="0" iyy="1.1e-09" iyz="0" izz="1.1e-09"/>
-		</inertial>
 		<xacro:insert_visu_RFinger22_link/>
 	</link>
@@ -89,8 +65,4 @@
 	</joint>
 	<link name="LFinger22_link">
-		<inertial>
-			<mass value="2e-06"/>
-			<inertia ixx="1.1e-09" ixy="0" ixz="0" iyy="1.1e-09" iyz="0" izz="1.1e-09"/>
-		</inertial>
 		<xacro:insert_visu_LFinger22_link/>
 	</link>
@@ -103,8 +75,4 @@
 	</joint>
 	<link name="RFinger21_link">
-		<inertial>
-			<mass value="2e-06"/>
-			<inertia ixx="1.1e-09" ixy="0" ixz="0" iyy="1.1e-09" iyz="0" izz="1.1e-09"/>
-		</inertial>
 		<xacro:insert_visu_RFinger21_link/>
 	</link>
@@ -117,8 +85,4 @@
 	</joint>
 	<link name="LFinger12_link">
-		<inertial>
-			<mass value="2e-06"/>
-			<inertia ixx="1.1e-09" ixy="0" ixz="0" iyy="1.1e-09" iyz="0" izz="1.1e-09"/>
-		</inertial>
 		<xacro:insert_visu_LFinger12_link/>
 	</link>
@@ -131,8 +95,4 @@
 	</joint>
 	<link name="RFinger23_link">
-		<inertial>
-			<mass value="2e-06"/>
-			<inertia ixx="1.1e-09" ixy="0" ixz="0" iyy="1.1e-09" iyz="0" izz="1.1e-09"/>
-		</inertial>
 		<xacro:insert_visu_RFinger23_link/>
 	</link>
@@ -145,8 +105,4 @@
 	</joint>
 	<link name="RFinger11_link">
-		<inertial>
-			<mass value="2e-06"/>
-			<inertia ixx="1.1e-09" ixy="0" ixz="0" iyy="1.1e-09" iyz="0" izz="1.1e-09"/>
-		</inertial>
 		<xacro:insert_visu_RFinger11_link/>
 	</link>
@@ -159,8 +115,4 @@
 	</joint>
 	<link name="LFinger23_link">
-		<inertial>
-			<mass value="2e-06"/>
-			<inertia ixx="1.1e-09" ixy="0" ixz="0" iyy="1.1e-09" iyz="0" izz="1.1e-09"/>
-		</inertial>
 		<xacro:insert_visu_LFinger23_link/>
 	</link>
@@ -173,8 +125,4 @@
 	</joint>
 	<link name="LThumb1_link">
-		<inertial>
-			<mass value="2e-06"/>
-			<inertia ixx="1.1e-09" ixy="0" ixz="0" iyy="1.1e-09" iyz="0" izz="1.1e-09"/>
-		</inertial>
 		<xacro:insert_visu_LThumb1_link/>
 	</link>
@@ -187,8 +135,4 @@
 	</joint>
 	<link name="RThumb1_link">
-		<inertial>
-			<mass value="2e-06"/>
-			<inertia ixx="1.1e-09" ixy="0" ixz="0" iyy="1.1e-09" iyz="0" izz="1.1e-09"/>
-		</inertial>
 		<xacro:insert_visu_RThumb1_link/>
 	</link>
@@ -201,8 +145,4 @@
 	</joint>
 	<link name="RThumb2_link">
-		<inertial>
-			<mass value="2e-06"/>
-			<inertia ixx="1.1e-09" ixy="0" ixz="0" iyy="1.1e-09" iyz="0" izz="1.1e-09"/>
-		</inertial>
 		<xacro:insert_visu_RThumb2_link/>
 	</link>
@@ -215,8 +155,4 @@
 	</joint>
 	<link name="LThumb2_link">
-		<inertial>
-			<mass value="2e-06"/>
-			<inertia ixx="1.1e-09" ixy="0" ixz="0" iyy="1.1e-09" iyz="0" izz="1.1e-09"/>
-		</inertial>
 		<xacro:insert_visu_LThumb2_link/>
 	</link>

File: nao_description/urdf/naoV33_generated_urdf/nao_sensors.xacro (robot description, xacro)
@@ -18,4 +18,10 @@
 		<axis xyz="0 0 0"/>
 	</joint>
+	<link name="CameraBottom_optical_frame"/>
+	<joint name="CameraBottom_optical_frame_joint" type="fixed">
+		<parent link="CameraBottom_frame"/>
+		<child link="CameraBottom_optical_frame"/>
+		<origin rpy="-1.57079632679 0 -1.57079632679" xyz="0 0 0"/>
+	</joint>
 	<link name="RFsrRR_frame"/>
 	<joint name="RFoot/FSR/RearRight_sensor_fixedjoint" type="fixed">
@@ -74,11 +80,4 @@
 		<axis xyz="0 0 0"/>
 	</joint>
-	<link name="LSonar_frame"/>
-	<joint name="Sonar/Right_sensor_fixedjoint" type="fixed">
-		<parent link="torso"/>
-		<child link="LSonar_frame"/>
-		<origin rpy="0.00478508 0.0436497 -0.392441" xyz="0.00558253 -0.0192068 0.0623853"/>
-		<axis xyz="0 0 0"/>
-	</joint>
 	<link name="HeadTouchFront_frame"/>
 	<joint name="Head/Touch/Front_sensor_fixedjoint" type="fixed">
@@ -130,4 +129,11 @@
 		<axis xyz="0 0 0"/>
 	</joint>
+	<link name="LSonar_frame"/>
+	<joint name="Sonar/Left_sensor_fixedjoint" type="fixed">
+		<parent link="torso"/>
+		<child link="LSonar_frame"/>
+		<origin rpy="-0.00478508 0.0436497 0.392441" xyz="0.00558253 0.0192068 0.0623853"/>
+		<axis xyz="0 0 0"/>
+	</joint>
 	<link name="MicroSurroundRight_frame"/>
 	<joint name="MicroRight_sensor_fixedjoint" type="fixed">
@@ -152,8 +158,8 @@
 	</joint>
 	<link name="RSonar_frame"/>
-	<joint name="Sonar/Left_sensor_fixedjoint" type="fixed">
+	<joint name="Sonar/Right_sensor_fixedjoint" type="fixed">
 		<parent link="torso"/>
 		<child link="RSonar_frame"/>
-		<origin rpy="-0.00478508 0.0436497 0.392441" xyz="0.00558253 0.0192068 0.0623853"/>
+		<origin rpy="0.00478508 0.0436497 -0.392441" xyz="0.00558253 -0.0192068 0.0623853"/>
 		<axis xyz="0 0 0"/>
 	</joint>
@@ -179,4 +185,10 @@
 		<axis xyz="0 0 0"/>
 	</joint>
+	<link name="CameraTop_optical_frame"/>
+	<joint name="CameraTop_optical_frame_joint" type="fixed">
+		<parent link="CameraTop_frame"/>
+		<child link="CameraTop_optical_frame"/>
+		<origin rpy="-1.57079632679 0 -1.57079632679" xyz="0 0 0"/>
+	</joint>
 	<link name="LInfraRed_frame"/>
 	<joint name="InfraredL_sensor_fixedjoint" type="fixed">

File: nao_description/urdf/naoV40_generated_urdf/nao_arms.xacro (robot description, xacro)
@@ -85,10 +85,5 @@
 		<limit effort="0.292" lower="0" upper="1.0" velocity="8.33"/>
 	</joint>
-	<link name="l_gripper">
-		<inertial>
-			<mass value="2e-06"/>
-			<inertia ixx="1.1e-09" ixy="0" ixz="0" iyy="1.1e-09" iyz="0" izz="1.1e-09"/>
-		</inertial>
-	</link>
+	<link name="l_gripper"/>
 	<joint name="RShoulderPitch" type="revolute">
 		<parent link="torso"/>
@@ -172,9 +167,4 @@
 		<limit effort="0.292" lower="0" upper="1.0" velocity="8.33"/>
 	</joint>
-	<link name="r_gripper">
-		<inertial>
-			<mass value="2e-06"/>
-			<inertia ixx="1.1e-09" ixy="0" ixz="0" iyy="1.1e-09" iyz="0" izz="1.1e-09"/>
-		</inertial>
-	</link>
+	<link name="r_gripper"/>
 </robot>

File: nao_description/urdf/naoV40_generated_urdf/nao_fingers.xacro (robot description, xacro)
@@ -5,8 +5,4 @@
 <robot name="naoH25V40" xmlns:xacro="http://www.ros.org/wiki/xacro">
 	<link name="RFinger13_link">
-		<inertial>
-			<mass value="2e-06"/>
-			<inertia ixx="1.1e-09" ixy="0" ixz="0" iyy="1.1e-09" iyz="0" izz="1.1e-09"/>
-		</inertial>
 		<xacro:insert_visu_RFinger13_link/>
 	</link>
@@ -19,8 +15,4 @@
 	</joint>
 	<link name="RFinger12_link">
-		<inertial>
-			<mass value="2e-06"/>
-			<inertia ixx="1.1e-09" ixy="0" ixz="0" iyy="1.1e-09" iyz="0" izz="1.1e-09"/>
-		</inertial>
 		<xacro:insert_visu_RFinger12_link/>
 	</link>
@@ -33,8 +25,4 @@
 	</joint>
 	<link name="LFinger21_link">
-		<inertial>
-			<mass value="2e-06"/>
-			<inertia ixx="1.1e-09" ixy="0" ixz="0" iyy="1.1e-09" iyz="0" izz="1.1e-09"/>
-		</inertial>
 		<xacro:insert_visu_LFinger21_link/>
 	</link>
@@ -47,8 +35,4 @@
 	</joint>
 	<link name="LFinger13_link">
-		<inertial>
-			<mass value="2e-06"/>
-			<inertia ixx="1.1e-09" ixy="0" ixz="0" iyy="1.1e-09" iyz="0" izz="1.1e-09"/>
-		</inertial>
 		<xacro:insert_visu_LFinger13_link/>
 	</link>
@@ -61,8 +45,4 @@
 	</joint>
 	<link name="LFinger11_link">
-		<inertial>
-			<mass value="2e-06"/>
-			<inertia ixx="1.1e-09" ixy="0" ixz="0" iyy="1.1e-09" iyz="0" izz="1.1e-09"/>
-		</inertial>
 		<xacro:insert_visu_LFinger11_link/>
 	</link>
@@ -75,8 +55,4 @@
 	</joint>
 	<link name="RFinger22_link">
-		<inertial>
-			<mass value="2e-06"/>
-			<inertia ixx="1.1e-09" ixy="0" ixz="0" iyy="1.1e-09" iyz="0" izz="1.1e-09"/>
-		</inertial>
 		<xacro:insert_visu_RFinger22_link/>
 	</link>
@@ -89,8 +65,4 @@
 	</joint>
 	<link name="LFinger22_link">
-		<inertial>
-			<mass value="2e-06"/>
-			<inertia ixx="1.1e-09" ixy="0" ixz="0" iyy="1.1e-09" iyz="0" izz="1.1e-09"/>
-		</inertial>
 		<xacro:insert_visu_LFinger22_link/>
 	</link>
@@ -103,8 +75,4 @@
 	</joint>
 	<link name="RFinger21_link">
-		<inertial>
-			<mass value="2e-06"/>
-			<inertia ixx="1.1e-09" ixy="0" ixz="0" iyy="1.1e-09" iyz="0" izz="1.1e-09"/>
-		</inertial>
 		<xacro:insert_visu_RFinger21_link/>
 	</link>
@@ -117,8 +85,4 @@
 	</joint>
 	<link name="LFinger12_link">
-		<inertial>
-			<mass value="2e-06"/>
-			<inertia ixx="1.1e-09" ixy="0" ixz="0" iyy="1.1e-09" iyz="0" izz="1.1e-09"/>
-		</inertial>
 		<xacro:insert_visu_LFinger12_link/>
 	</link>
@@ -131,8 +95,4 @@
 	</joint>
 	<link name="RFinger23_link">
-		<inertial>
-			<mass value="2e-06"/>
-			<inertia ixx="1.1e-09" ixy="0" ixz="0" iyy="1.1e-09" iyz="0" izz="1.1e-09"/>
-		</inertial>
 		<xacro:insert_visu_RFinger23_link/>
 	</link>
@@ -145,8 +105,4 @@
 	</joint>
 	<link name="RFinger11_link">
-		<inertial>
-			<mass value="2e-06"/>
-			<inertia ixx="1.1e-09" ixy="0" ixz="0" iyy="1.1e-09" iyz="0" izz="1.1e-09"/>
-		</inertial>
 		<xacro:insert_visu_RFinger11_link/>
 	</link>
@@ -159,8 +115,4 @@
 	</joint>
 	<link name="LFinger23_link">
-		<inertial>
-			<mass value="2e-06"/>
-			<inertia ixx="1.1e-09" ixy="0" ixz="0" iyy="1.1e-09" iyz="0" izz="1.1e-09"/>
-		</inertial>
 		<xacro:insert_visu_LFinger23_link/>
 	</link>
@@ -173,8 +125,4 @@
 	</joint>
 	<link name="LThumb1_link">
-		<inertial>
-			<mass value="2e-06"/>
-			<inertia ixx="1.1e-09" ixy="0" ixz="0" iyy="1.1e-09" iyz="0" izz="1.1e-09"/>
-		</inertial>
 		<xacro:insert_visu_LThumb1_link/>
 	</link>
@@ -187,8 +135,4 @@
 	</joint>
 	<link name="RThumb1_link">
-		<inertial>
-			<mass value="2e-06"/>
-			<inertia ixx="1.1e-09" ixy="0" ixz="0" iyy="1.1e-09" iyz="0" izz="1.1e-09"/>
-		</inertial>
 		<xacro:insert_visu_RThumb1_link/>
 	</link>
@@ -201,8 +145,4 @@
 	</joint>
 	<link name="RThumb2_link">
-		<inertial>
-			<mass value="2e-06"/>
-			<inertia ixx="1.1e-09" ixy="0" ixz="0" iyy="1.1e-09" iyz="0" izz="1.1e-09"/>
-		</inertial>
 		<xacro:insert_visu_RThumb2_link/>
 	</link>
@@ -215,8 +155,4 @@
 	</joint>
 	<link name="LThumb2_link">
-		<inertial>
-			<mass value="2e-06"/>
-			<inertia ixx="1.1e-09" ixy="0" ixz="0" iyy="1.1e-09" iyz="0" izz="1.1e-09"/>
-		</inertial>
 		<xacro:insert_visu_LThumb2_link/>
 	</link>
