Commit message: properly fix 535d34474d9f64ddb60f6f163656c10fcdf92774 The automatic generator was used to generate inertia

File: nao_description/urdf/naoV32_generated_urdf/nao_arms.xacro (robot description, xacro)
@@ -86,8 +86,8 @@
 	</joint>
 	<link name="l_gripper">
-	  <inertial>
-	    <mass value="2e-06"/>
-	    <inertia ixx="1.1e-09" ixy="0" ixz="0" iyy="1.1e-09" iyz="0" izz="1.1e-09"/>
-	  </inertial>
+		<inertial>
+			<mass value="2e-06"/>
+			<inertia ixx="1.1e-09" ixy="0" ixz="0" iyy="1.1e-09" iyz="0" izz="1.1e-09"/>
+		</inertial>
 	</link>
 	<joint name="RShoulderPitch" type="revolute">
@@ -173,8 +173,8 @@
 	</joint>
 	<link name="r_gripper">
-	  <inertial>
-	    <mass value="2e-06"/>
-	    <inertia ixx="1.1e-09" ixy="0" ixz="0" iyy="1.1e-09" iyz="0" izz="1.1e-09"/>
-	  </inertial>
+		<inertial>
+			<mass value="2e-06"/>
+			<inertia ixx="1.1e-09" ixy="0" ixz="0" iyy="1.1e-09" iyz="0" izz="1.1e-09"/>
+		</inertial>
 	</link>
 </robot>

File: nao_description/urdf/naoV32_generated_urdf/nao_fingers.xacro (robot description, xacro)
@@ -5,9 +5,9 @@
 <robot name="naoH25V32" xmlns:xacro="http://www.ros.org/wiki/xacro">
 	<link name="RFinger13_link">
-	    <xacro:insert_visu_RFinger13_link/>
-            <inertial>
-	        <mass value="2e-06"/>
-	        <inertia ixx="1.1e-09" ixy="0" ixz="0" iyy="1.1e-09" iyz="0" izz="1.1e-09"/>
-	    </inertial>
+		<inertial>
+			<mass value="2e-06"/>
+			<inertia ixx="1.1e-09" ixy="0" ixz="0" iyy="1.1e-09" iyz="0" izz="1.1e-09"/>
+		</inertial>
+		<xacro:insert_visu_RFinger13_link/>
 	</link>
 	<joint name="RFinger13" type="continuous">
@@ -19,9 +19,9 @@
 	</joint>
 	<link name="RFinger12_link">
+		<inertial>
+			<mass value="2e-06"/>
+			<inertia ixx="1.1e-09" ixy="0" ixz="0" iyy="1.1e-09" iyz="0" izz="1.1e-09"/>
+		</inertial>
 		<xacro:insert_visu_RFinger12_link/>
-            <inertial>
-	        <mass value="2e-06"/>
-	        <inertia ixx="1.1e-09" ixy="0" ixz="0" iyy="1.1e-09" iyz="0" izz="1.1e-09"/>
-	    </inertial>
 	</link>
 	<joint name="RFinger12" type="continuous">
@@ -33,9 +33,9 @@
 	</joint>
 	<link name="LFinger21_link">
+		<inertial>
+			<mass value="2e-06"/>
+			<inertia ixx="1.1e-09" ixy="0" ixz="0" iyy="1.1e-09" iyz="0" izz="1.1e-09"/>
+		</inertial>
 		<xacro:insert_visu_LFinger21_link/>
-            <inertial>
-	        <mass value="2e-06"/>
-	        <inertia ixx="1.1e-09" ixy="0" ixz="0" iyy="1.1e-09" iyz="0" izz="1.1e-09"/>
-	    </inertial>
 	</link>
 	<joint name="LFinger21" type="continuous">
@@ -47,9 +47,9 @@
 	</joint>
 	<link name="LFinger13_link">
+		<inertial>
+			<mass value="2e-06"/>
+			<inertia ixx="1.1e-09" ixy="0" ixz="0" iyy="1.1e-09" iyz="0" izz="1.1e-09"/>
+		</inertial>
 		<xacro:insert_visu_LFinger13_link/>
-            <inertial>
-	        <mass value="2e-06"/>
-	        <inertia ixx="1.1e-09" ixy="0" ixz="0" iyy="1.1e-09" iyz="0" izz="1.1e-09"/>
-	    </inertial>
 	</link>
 	<joint name="LFinger13" type="continuous">
@@ -61,9 +61,9 @@
 	</joint>
 	<link name="LFinger11_link">
+		<inertial>
+			<mass value="2e-06"/>
+			<inertia ixx="1.1e-09" ixy="0" ixz="0" iyy="1.1e-09" iyz="0" izz="1.1e-09"/>
+		</inertial>
 		<xacro:insert_visu_LFinger11_link/>
-            <inertial>
-	        <mass value="2e-06"/>
-	        <inertia ixx="1.1e-09" ixy="0" ixz="0" iyy="1.1e-09" iyz="0" izz="1.1e-09"/>
-	    </inertial>
 	</link>
 	<joint name="LFinger11" type="continuous">
@@ -75,9 +75,9 @@
 	</joint>
 	<link name="RFinger22_link">
+		<inertial>
+			<mass value="2e-06"/>
+			<inertia ixx="1.1e-09" ixy="0" ixz="0" iyy="1.1e-09" iyz="0" izz="1.1e-09"/>
+		</inertial>
 		<xacro:insert_visu_RFinger22_link/>
-            <inertial>
-	        <mass value="2e-06"/>
-	        <inertia ixx="1.1e-09" ixy="0" ixz="0" iyy="1.1e-09" iyz="0" izz="1.1e-09"/>
-	    </inertial>
 	</link>
 	<joint name="RFinger22" type="continuous">
@@ -89,9 +89,9 @@
 	</joint>
 	<link name="LFinger22_link">
+		<inertial>
+			<mass value="2e-06"/>
+			<inertia ixx="1.1e-09" ixy="0" ixz="0" iyy="1.1e-09" iyz="0" izz="1.1e-09"/>
+		</inertial>
 		<xacro:insert_visu_LFinger22_link/>
-            <inertial>
-	        <mass value="2e-06"/>
-	        <inertia ixx="1.1e-09" ixy="0" ixz="0" iyy="1.1e-09" iyz="0" izz="1.1e-09"/>
-	    </inertial>
 	</link>
 	<joint name="LFinger22" type="continuous">
@@ -103,9 +103,9 @@
 	</joint>
 	<link name="RFinger21_link">
+		<inertial>
+			<mass value="2e-06"/>
+			<inertia ixx="1.1e-09" ixy="0" ixz="0" iyy="1.1e-09" iyz="0" izz="1.1e-09"/>
+		</inertial>
 		<xacro:insert_visu_RFinger21_link/>
-            <inertial>
-	        <mass value="2e-06"/>
-	        <inertia ixx="1.1e-09" ixy="0" ixz="0" iyy="1.1e-09" iyz="0" izz="1.1e-09"/>
-	    </inertial>
 	</link>
 	<joint name="RFinger21" type="continuous">
@@ -117,9 +117,9 @@
 	</joint>
 	<link name="LFinger12_link">
+		<inertial>
+			<mass value="2e-06"/>
+			<inertia ixx="1.1e-09" ixy="0" ixz="0" iyy="1.1e-09" iyz="0" izz="1.1e-09"/>
+		</inertial>
 		<xacro:insert_visu_LFinger12_link/>
-            <inertial>
-	        <mass value="2e-06"/>
-	        <inertia ixx="1.1e-09" ixy="0" ixz="0" iyy="1.1e-09" iyz="0" izz="1.1e-09"/>
-	    </inertial>
 	</link>
 	<joint name="LFinger12" type="continuous">
@@ -131,9 +131,9 @@
 	</joint>
 	<link name="RFinger23_link">
+		<inertial>
+			<mass value="2e-06"/>
+			<inertia ixx="1.1e-09" ixy="0" ixz="0" iyy="1.1e-09" iyz="0" izz="1.1e-09"/>
+		</inertial>
 		<xacro:insert_visu_RFinger23_link/>
-            <inertial>
-	        <mass value="2e-06"/>
-	        <inertia ixx="1.1e-09" ixy="0" ixz="0" iyy="1.1e-09" iyz="0" izz="1.1e-09"/>
-	    </inertial>
 	</link>
 	<joint name="RFinger23" type="continuous">
@@ -145,9 +145,9 @@
 	</joint>
 	<link name="RFinger11_link">
+		<inertial>
+			<mass value="2e-06"/>
+			<inertia ixx="1.1e-09" ixy="0" ixz="0" iyy="1.1e-09" iyz="0" izz="1.1e-09"/>
+		</inertial>
 		<xacro:insert_visu_RFinger11_link/>
-            <inertial>
-	        <mass value="2e-06"/>
-	        <inertia ixx="1.1e-09" ixy="0" ixz="0" iyy="1.1e-09" iyz="0" izz="1.1e-09"/>
-	    </inertial>
 	</link>
 	<joint name="RFinger11" type="continuous">
@@ -159,9 +159,9 @@
 	</joint>
 	<link name="LFinger23_link">
+		<inertial>
+			<mass value="2e-06"/>
+			<inertia ixx="1.1e-09" ixy="0" ixz="0" iyy="1.1e-09" iyz="0" izz="1.1e-09"/>
+		</inertial>
 		<xacro:insert_visu_LFinger23_link/>
-            <inertial>
-	        <mass value="2e-06"/>
-	        <inertia ixx="1.1e-09" ixy="0" ixz="0" iyy="1.1e-09" iyz="0" izz="1.1e-09"/>
-	    </inertial>
 	</link>
 	<joint name="LFinger23" type="continuous">
@@ -173,9 +173,9 @@
 	</joint>
 	<link name="LThumb1_link">
+		<inertial>
+			<mass value="2e-06"/>
+			<inertia ixx="1.1e-09" ixy="0" ixz="0" iyy="1.1e-09" iyz="0" izz="1.1e-09"/>
+		</inertial>
 		<xacro:insert_visu_LThumb1_link/>
-            <inertial>
-	        <mass value="2e-06"/>
-	        <inertia ixx="1.1e-09" ixy="0" ixz="0" iyy="1.1e-09" iyz="0" izz="1.1e-09"/>
-	    </inertial>
 	</link>
 	<joint name="LThumb1" type="continuous">
@@ -187,9 +187,9 @@
 	</joint>
 	<link name="RThumb1_link">
+		<inertial>
+			<mass value="2e-06"/>
+			<inertia ixx="1.1e-09" ixy="0" ixz="0" iyy="1.1e-09" iyz="0" izz="1.1e-09"/>
+		</inertial>
 		<xacro:insert_visu_RThumb1_link/>
-            <inertial>
-	        <mass value="2e-06"/>
-	        <inertia ixx="1.1e-09" ixy="0" ixz="0" iyy="1.1e-09" iyz="0" izz="1.1e-09"/>
-	    </inertial>
 	</link>
 	<joint name="RThumb1" type="continuous">
@@ -201,9 +201,9 @@
 	</joint>
 	<link name="RThumb2_link">
+		<inertial>
+			<mass value="2e-06"/>
+			<inertia ixx="1.1e-09" ixy="0" ixz="0" iyy="1.1e-09" iyz="0" izz="1.1e-09"/>
+		</inertial>
 		<xacro:insert_visu_RThumb2_link/>
-            <inertial>
-	        <mass value="2e-06"/>
-	        <inertia ixx="1.1e-09" ixy="0" ixz="0" iyy="1.1e-09" iyz="0" izz="1.1e-09"/>
-	    </inertial>
 	</link>
 	<joint name="RThumb2" type="continuous">
@@ -215,9 +215,9 @@
 	</joint>
 	<link name="LThumb2_link">
+		<inertial>
+			<mass value="2e-06"/>
+			<inertia ixx="1.1e-09" ixy="0" ixz="0" iyy="1.1e-09" iyz="0" izz="1.1e-09"/>
+		</inertial>
 		<xacro:insert_visu_LThumb2_link/>
-            <inertial>
-	        <mass value="2e-06"/>
-	        <inertia ixx="1.1e-09" ixy="0" ixz="0" iyy="1.1e-09" iyz="0" izz="1.1e-09"/>
-	    </inertial>
 	</link>
 	<joint name="LThumb2" type="continuous">

File: nao_description/urdf/naoV33_generated_urdf/nao_arms.xacro (robot description, xacro)
@@ -86,8 +86,8 @@
 	</joint>
 	<link name="l_gripper">
-	  <inertial>
-	    <mass value="2e-06"/>
-	    <inertia ixx="1.1e-09" ixy="0" ixz="0" iyy="1.1e-09" iyz="0" izz="1.1e-09"/>
-	  </inertial>
+		<inertial>
+			<mass value="2e-06"/>
+			<inertia ixx="1.1e-09" ixy="0" ixz="0" iyy="1.1e-09" iyz="0" izz="1.1e-09"/>
+		</inertial>
 	</link>
 	<joint name="RShoulderPitch" type="revolute">
@@ -173,8 +173,8 @@
 	</joint>
 	<link name="r_gripper">
-	  <inertial>
-	    <mass value="2e-06"/>
-	    <inertia ixx="1.1e-09" ixy="0" ixz="0" iyy="1.1e-09" iyz="0" izz="1.1e-09"/>
-	  </inertial>
+		<inertial>
+			<mass value="2e-06"/>
+			<inertia ixx="1.1e-09" ixy="0" ixz="0" iyy="1.1e-09" iyz="0" izz="1.1e-09"/>
+		</inertial>
 	</link>
 </robot>

File: nao_description/urdf/naoV33_generated_urdf/nao_fingers.xacro (robot description, xacro)
@@ -5,9 +5,9 @@
 <robot name="naoH25V33" xmlns:xacro="http://www.ros.org/wiki/xacro">
 	<link name="RFinger13_link">
-	    <xacro:insert_visu_RFinger13_link/>
-            <inertial>
-	        <mass value="2e-06"/>
-	        <inertia ixx="1.1e-09" ixy="0" ixz="0" iyy="1.1e-09" iyz="0" izz="1.1e-09"/>
-	    </inertial>
+		<inertial>
+			<mass value="2e-06"/>
+			<inertia ixx="1.1e-09" ixy="0" ixz="0" iyy="1.1e-09" iyz="0" izz="1.1e-09"/>
+		</inertial>
+		<xacro:insert_visu_RFinger13_link/>
 	</link>
 	<joint name="RFinger13" type="continuous">
@@ -19,9 +19,9 @@
 	</joint>
 	<link name="RFinger12_link">
+		<inertial>
+			<mass value="2e-06"/>
+			<inertia ixx="1.1e-09" ixy="0" ixz="0" iyy="1.1e-09" iyz="0" izz="1.1e-09"/>
+		</inertial>
 		<xacro:insert_visu_RFinger12_link/>
-            <inertial>
-	        <mass value="2e-06"/>
-	        <inertia ixx="1.1e-09" ixy="0" ixz="0" iyy="1.1e-09" iyz="0" izz="1.1e-09"/>
-	    </inertial>
 	</link>
 	<joint name="RFinger12" type="continuous">
@@ -33,9 +33,9 @@
 	</joint>
 	<link name="LFinger21_link">
+		<inertial>
+			<mass value="2e-06"/>
+			<inertia ixx="1.1e-09" ixy="0" ixz="0" iyy="1.1e-09" iyz="0" izz="1.1e-09"/>
+		</inertial>
 		<xacro:insert_visu_LFinger21_link/>
-            <inertial>
-	        <mass value="2e-06"/>
-	        <inertia ixx="1.1e-09" ixy="0" ixz="0" iyy="1.1e-09" iyz="0" izz="1.1e-09"/>
-	    </inertial>
 	</link>
 	<joint name="LFinger21" type="continuous">
@@ -47,9 +47,9 @@
 	</joint>
 	<link name="LFinger13_link">
+		<inertial>
+			<mass value="2e-06"/>
+			<inertia ixx="1.1e-09" ixy="0" ixz="0" iyy="1.1e-09" iyz="0" izz="1.1e-09"/>
+		</inertial>
 		<xacro:insert_visu_LFinger13_link/>
-            <inertial>
-	        <mass value="2e-06"/>
-	        <inertia ixx="1.1e-09" ixy="0" ixz="0" iyy="1.1e-09" iyz="0" izz="1.1e-09"/>
-	    </inertial>
 	</link>
 	<joint name="LFinger13" type="continuous">
@@ -61,9 +61,9 @@
 	</joint>
 	<link name="LFinger11_link">
+		<inertial>
+			<mass value="2e-06"/>
+			<inertia ixx="1.1e-09" ixy="0" ixz="0" iyy="1.1e-09" iyz="0" izz="1.1e-09"/>
+		</inertial>
 		<xacro:insert_visu_LFinger11_link/>
-            <inertial>
-	        <mass value="2e-06"/>
-	        <inertia ixx="1.1e-09" ixy="0" ixz="0" iyy="1.1e-09" iyz="0" izz="1.1e-09"/>
-	    </inertial>
 	</link>
 	<joint name="LFinger11" type="continuous">
@@ -75,9 +75,9 @@
 	</joint>
 	<link name="RFinger22_link">
+		<inertial>
+			<mass value="2e-06"/>
+			<inertia ixx="1.1e-09" ixy="0" ixz="0" iyy="1.1e-09" iyz="0" izz="1.1e-09"/>
+		</inertial>
 		<xacro:insert_visu_RFinger22_link/>
-            <inertial>
-	        <mass value="2e-06"/>
-	        <inertia ixx="1.1e-09" ixy="0" ixz="0" iyy="1.1e-09" iyz="0" izz="1.1e-09"/>
-	    </inertial>
 	</link>
 	<joint name="RFinger22" type="continuous">
@@ -89,9 +89,9 @@
 	</joint>
 	<link name="LFinger22_link">
+		<inertial>
+			<mass value="2e-06"/>
+			<inertia ixx="1.1e-09" ixy="0" ixz="0" iyy="1.1e-09" iyz="0" izz="1.1e-09"/>
+		</inertial>
 		<xacro:insert_visu_LFinger22_link/>
-            <inertial>
-	        <mass value="2e-06"/>
-	        <inertia ixx="1.1e-09" ixy="0" ixz="0" iyy="1.1e-09" iyz="0" izz="1.1e-09"/>
-	    </inertial>
 	</link>
 	<joint name="LFinger22" type="continuous">
@@ -103,9 +103,9 @@
 	</joint>
 	<link name="RFinger21_link">
+		<inertial>
+			<mass value="2e-06"/>
+			<inertia ixx="1.1e-09" ixy="0" ixz="0" iyy="1.1e-09" iyz="0" izz="1.1e-09"/>
+		</inertial>
 		<xacro:insert_visu_RFinger21_link/>
-            <inertial>
-	        <mass value="2e-06"/>
-	        <inertia ixx="1.1e-09" ixy="0" ixz="0" iyy="1.1e-09" iyz="0" izz="1.1e-09"/>
-	    </inertial>
 	</link>
 	<joint name="RFinger21" type="continuous">
@@ -117,9 +117,9 @@
 	</joint>
 	<link name="LFinger12_link">
+		<inertial>
+			<mass value="2e-06"/>
+			<inertia ixx="1.1e-09" ixy="0" ixz="0" iyy="1.1e-09" iyz="0" izz="1.1e-09"/>
+		</inertial>
 		<xacro:insert_visu_LFinger12_link/>
-            <inertial>
-	        <mass value="2e-06"/>
-	        <inertia ixx="1.1e-09" ixy="0" ixz="0" iyy="1.1e-09" iyz="0" izz="1.1e-09"/>
-	    </inertial>
 	</link>
 	<joint name="LFinger12" type="continuous">
@@ -131,9 +131,9 @@
 	</joint>
 	<link name="RFinger23_link">
+		<inertial>
+			<mass value="2e-06"/>
+			<inertia ixx="1.1e-09" ixy="0" ixz="0" iyy="1.1e-09" iyz="0" izz="1.1e-09"/>
+		</inertial>
 		<xacro:insert_visu_RFinger23_link/>
-            <inertial>
-	        <mass value="2e-06"/>
-	        <inertia ixx="1.1e-09" ixy="0" ixz="0" iyy="1.1e-09" iyz="0" izz="1.1e-09"/>
-	    </inertial>
 	</link>
 	<joint name="RFinger23" type="continuous">
@@ -145,9 +145,9 @@
 	</joint>
 	<link name="RFinger11_link">
+		<inertial>
+			<mass value="2e-06"/>
+			<inertia ixx="1.1e-09" ixy="0" ixz="0" iyy="1.1e-09" iyz="0" izz="1.1e-09"/>
+		</inertial>
 		<xacro:insert_visu_RFinger11_link/>
-            <inertial>
-	        <mass value="2e-06"/>
-	        <inertia ixx="1.1e-09" ixy="0" ixz="0" iyy="1.1e-09" iyz="0" izz="1.1e-09"/>
-	    </inertial>
 	</link>
 	<joint name="RFinger11" type="continuous">
@@ -159,9 +159,9 @@
 	</joint>
 	<link name="LFinger23_link">
+		<inertial>
+			<mass value="2e-06"/>
+			<inertia ixx="1.1e-09" ixy="0" ixz="0" iyy="1.1e-09" iyz="0" izz="1.1e-09"/>
+		</inertial>
 		<xacro:insert_visu_LFinger23_link/>
-            <inertial>
-	        <mass value="2e-06"/>
-	        <inertia ixx="1.1e-09" ixy="0" ixz="0" iyy="1.1e-09" iyz="0" izz="1.1e-09"/>
-	    </inertial>
 	</link>
 	<joint name="LFinger23" type="continuous">
@@ -173,9 +173,9 @@
 	</joint>
 	<link name="LThumb1_link">
+		<inertial>
+			<mass value="2e-06"/>
+			<inertia ixx="1.1e-09" ixy="0" ixz="0" iyy="1.1e-09" iyz="0" izz="1.1e-09"/>
+		</inertial>
 		<xacro:insert_visu_LThumb1_link/>
-            <inertial>
-	        <mass value="2e-06"/>
-	        <inertia ixx="1.1e-09" ixy="0" ixz="0" iyy="1.1e-09" iyz="0" izz="1.1e-09"/>
-	    </inertial>
 	</link>
 	<joint name="LThumb1" type="continuous">
@@ -187,9 +187,9 @@
 	</joint>
 	<link name="RThumb1_link">
+		<inertial>
+			<mass value="2e-06"/>
+			<inertia ixx="1.1e-09" ixy="0" ixz="0" iyy="1.1e-09" iyz="0" izz="1.1e-09"/>
+		</inertial>
 		<xacro:insert_visu_RThumb1_link/>
-            <inertial>
-	        <mass value="2e-06"/>
-	        <inertia ixx="1.1e-09" ixy="0" ixz="0" iyy="1.1e-09" iyz="0" izz="1.1e-09"/>
-	    </inertial>
 	</link>
 	<joint name="RThumb1" type="continuous">
@@ -201,9 +201,9 @@
 	</joint>
 	<link name="RThumb2_link">
+		<inertial>
+			<mass value="2e-06"/>
+			<inertia ixx="1.1e-09" ixy="0" ixz="0" iyy="1.1e-09" iyz="0" izz="1.1e-09"/>
+		</inertial>
 		<xacro:insert_visu_RThumb2_link/>
-            <inertial>
-	        <mass value="2e-06"/>
-	        <inertia ixx="1.1e-09" ixy="0" ixz="0" iyy="1.1e-09" iyz="0" izz="1.1e-09"/>
-	    </inertial>
 	</link>
 	<joint name="RThumb2" type="continuous">
@@ -215,9 +215,9 @@
 	</joint>
 	<link name="LThumb2_link">
+		<inertial>
+			<mass value="2e-06"/>
+			<inertia ixx="1.1e-09" ixy="0" ixz="0" iyy="1.1e-09" iyz="0" izz="1.1e-09"/>
+		</inertial>
 		<xacro:insert_visu_LThumb2_link/>
-            <inertial>
-	        <mass value="2e-06"/>
-	        <inertia ixx="1.1e-09" ixy="0" ixz="0" iyy="1.1e-09" iyz="0" izz="1.1e-09"/>
-	    </inertial>
 	</link>
 	<joint name="LThumb2" type="continuous">

File: nao_description/urdf/naoV40_generated_urdf/nao_arms.xacro (robot description, xacro)
@@ -86,8 +86,8 @@
 	</joint>
 	<link name="l_gripper">
-	  <inertial>
-	    <mass value="2e-06"/>
-	    <inertia ixx="1.1e-09" ixy="0" ixz="0" iyy="1.1e-09" iyz="0" izz="1.1e-09"/>
-	  </inertial>
+		<inertial>
+			<mass value="2e-06"/>
+			<inertia ixx="1.1e-09" ixy="0" ixz="0" iyy="1.1e-09" iyz="0" izz="1.1e-09"/>
+		</inertial>
 	</link>
 	<joint name="RShoulderPitch" type="revolute">
@@ -173,8 +173,8 @@
 	</joint>
 	<link name="r_gripper">
-	  <inertial>
-	    <mass value="2e-06"/>
-	    <inertia ixx="1.1e-09" ixy="0" ixz="0" iyy="1.1e-09" iyz="0" izz="1.1e-09"/>
-	  </inertial>
+		<inertial>
+			<mass value="2e-06"/>
+			<inertia ixx="1.1e-09" ixy="0" ixz="0" iyy="1.1e-09" iyz="0" izz="1.1e-09"/>
+		</inertial>
 	</link>
 </robot>
