Commit message: update full .urdf file using xacro

File: nao_description/urdf/naoV32_generated_urdf/nao.urdf (robot description, URDF)
Before this commit: robot naoH25V32, 75 links, 74 joints
Links:
- added link CameraBottom_optical_frame
- added link CameraTop_optical_frame
Joints:
- added joint CameraBottom_optical_frame_joint: type fixed, parent CameraBottom_frame, child CameraBottom_optical_frame, origin xyz=0 0 0 rpy=-1.57079632679 0 -1.57079632679
- added joint CameraTop_optical_frame_joint: type fixed, parent CameraTop_frame, child CameraTop_optical_frame, origin xyz=0 0 0 rpy=-1.57079632679 0 -1.57079632679
- joint Sonar/Left_sensor_fixedjoint: child RSonar_frame -> LSonar_frame
- joint Sonar/Right_sensor_fixedjoint: child LSonar_frame -> RSonar_frame

File: nao_description/urdf/naoV33_generated_urdf/nao.urdf (robot description, URDF)
Before this commit: robot naoH25V33, 81 links, 80 joints
Links:
- added link CameraBottom_optical_frame
- added link CameraTop_optical_frame
Joints:
- added joint CameraBottom_optical_frame_joint: type fixed, parent CameraBottom_frame, child CameraBottom_optical_frame, origin xyz=0 0 0 rpy=-1.57079632679 0 -1.57079632679
- added joint CameraTop_optical_frame_joint: type fixed, parent CameraTop_frame, child CameraTop_optical_frame, origin xyz=0 0 0 rpy=-1.57079632679 0 -1.57079632679
- joint Sonar/Left_sensor_fixedjoint: child RSonar_frame -> LSonar_frame
- joint Sonar/Right_sensor_fixedjoint: child LSonar_frame -> RSonar_frame

File: nao_description/urdf/naoV40_generated_urdf/nao.urdf (robot description, URDF)
Before this commit: robot naoH25V40, 83 links, 82 joints
Links:
- link LFinger11_link: mass None -> 2e-06
- link LFinger12_link: mass None -> 2e-06
- link LFinger13_link: mass None -> 2e-06
- link LFinger21_link: mass None -> 2e-06
- link LFinger22_link: mass None -> 2e-06
- link LFinger23_link: mass None -> 2e-06
- link LThumb1_link: mass None -> 2e-06
- link LThumb2_link: mass None -> 2e-06
- link RFinger11_link: mass None -> 2e-06
- link RFinger12_link: mass None -> 2e-06
- link RFinger13_link: mass None -> 2e-06
- link RFinger21_link: mass None -> 2e-06
- link RFinger22_link: mass None -> 2e-06
- link RFinger23_link: mass None -> 2e-06
- link RThumb1_link: mass None -> 2e-06
- link RThumb2_link: mass None -> 2e-06
- link l_gripper: mass None -> 2e-06
- link r_gripper: mass None -> 2e-06

File: nao_description/urdf/naoV50_generated_urdf/nao.urdf (robot description, URDF)
Before this commit: robot naoH25V50, 77 links, 76 joints
Links:
- added link CameraBottom_optical_frame
- added link CameraTop_optical_frame
Joints:
- added joint CameraBottom_optical_frame_joint: type fixed, parent CameraBottom_frame, child CameraBottom_optical_frame, origin xyz=0 0 0 rpy=-1.57079632679 0 -1.57079632679
- added joint CameraTop_optical_frame_joint: type fixed, parent CameraTop_frame, child CameraTop_optical_frame, origin xyz=0 0 0 rpy=-1.57079632679 0 -1.57079632679
- joint Sonar/Left_sensor_fixedjoint: child RSonar_frame -> LSonar_frame
- joint Sonar/Right_sensor_fixedjoint: child LSonar_frame -> RSonar_frame

Commit message: generated urdf with simulated FSR

File: nao_description/urdf/naoV32_generated_urdf/nao.urdf (robot description, URDF)
Before this commit: robot naoH25V32, 77 links, 76 joints
Links:
- link LFsrFL_frame: mass None -> 2e-06; geometry collision box size=0.01 0.01 0.005
- link LFsrFR_frame: mass None -> 2e-06; geometry collision box size=0.01 0.01 0.005
- link LFsrRL_frame: mass None -> 2e-06; geometry collision box size=0.01 0.01 0.005
- link LFsrRR_frame: mass None -> 2e-06; geometry collision box size=0.01 0.01 0.005
- link RFsrFL_frame: mass None -> 2e-06; geometry collision box size=0.01 0.01 0.005
- link RFsrFR_frame: mass None -> 2e-06; geometry collision box size=0.01 0.01 0.005
- link RFsrRL_frame: mass None -> 2e-06; geometry collision box size=0.01 0.01 0.005
- link RFsrRR_frame: mass None -> 2e-06; geometry collision box size=0.01 0.01 0.005
Joints:
- removed joint CameraBottom_optical_frame_joint
- removed joint CameraTop_optical_frame_joint
- added joint CameraBottom_optical_frame_fixedjoint: type fixed, parent CameraBottom_frame, child CameraBottom_optical_frame, origin xyz=0 0 0 rpy=-1.57079632679 0 -1.57079632679
- added joint CameraTop_optical_frame_fixedjoint: type fixed, parent CameraTop_frame, child CameraTop_optical_frame, origin xyz=0 0 0 rpy=-1.57079632679 0 -1.57079632679

File: nao_description/urdf/naoV32_generated_urdf/nao_robot.xacro (robot description, xacro)
@@ -3,8 +3,8 @@
  ****** File automatically generated by generate_urdf.py script ******
  *********************************************************************-->
-<robot name="naoH25V32" xmlns:xacro="http://www.ros.org/wiki/xacro">
+<robot name="NaoH25V32" xmlns:xacro="http://www.ros.org/wiki/xacro">
 	<xacro:include filename="nao_visual_collisions.xacro"/>
-	<xacro:include filename="naoTransmission.xacro"/>
-	<xacro:include filename="naoGazebo.xacro"/>
+  <xacro:include filename="naoTransmission.xacro"/>
+  <xacro:include filename="naoGazebo.xacro"/>
 	<xacro:include filename="nao_head.xacro"/>
 	<xacro:include filename="nao_legs.xacro"/>

File: nao_description/urdf/naoV33_generated_urdf/nao.urdf (robot description, URDF)
Before this commit: robot naoH25V33, 83 links, 82 joints
Links:
- link LFsrFL_frame: mass None -> 2e-06; geometry collision box size=0.01 0.01 0.005
- link LFsrFR_frame: mass None -> 2e-06; geometry collision box size=0.01 0.01 0.005
- link LFsrRL_frame: mass None -> 2e-06; geometry collision box size=0.01 0.01 0.005
- link LFsrRR_frame: mass None -> 2e-06; geometry collision box size=0.01 0.01 0.005
- link RFsrFL_frame: mass None -> 2e-06; geometry collision box size=0.01 0.01 0.005
- link RFsrFR_frame: mass None -> 2e-06; geometry collision box size=0.01 0.01 0.005
- link RFsrRL_frame: mass None -> 2e-06; geometry collision box size=0.01 0.01 0.005
- link RFsrRR_frame: mass None -> 2e-06; geometry collision box size=0.01 0.01 0.005
Joints:
- removed joint CameraBottom_optical_frame_joint
- removed joint CameraTop_optical_frame_joint
- added joint CameraBottom_optical_frame_fixedjoint: type fixed, parent CameraBottom_frame, child CameraBottom_optical_frame, origin xyz=0 0 0 rpy=-1.57079632679 0 -1.57079632679
- added joint CameraTop_optical_frame_fixedjoint: type fixed, parent CameraTop_frame, child CameraTop_optical_frame, origin xyz=0 0 0 rpy=-1.57079632679 0 -1.57079632679

File: nao_description/urdf/naoV33_generated_urdf/nao_robot.xacro (robot description, xacro)
@@ -3,5 +3,5 @@
  ****** File automatically generated by generate_urdf.py script ******
  *********************************************************************-->
-<robot name="naoH25V33" xmlns:xacro="http://www.ros.org/wiki/xacro">
+<robot name="NaoH25V33" xmlns:xacro="http://www.ros.org/wiki/xacro">
 	<xacro:include filename="nao_visual_collisions.xacro"/>
 	<xacro:include filename="naoTransmission.xacro"/>

File: nao_description/urdf/naoV40_generated_urdf/nao.urdf (robot description, URDF)
Before this commit: robot naoH25V40, 83 links, 82 joints
Links:
- link LFsrFL_frame: mass None -> 2e-06; geometry collision box size=0.01 0.01 0.005
- link LFsrFR_frame: mass None -> 2e-06; geometry collision box size=0.01 0.01 0.005
- link LFsrRL_frame: mass None -> 2e-06; geometry collision box size=0.01 0.01 0.005
- link LFsrRR_frame: mass None -> 2e-06; geometry collision box size=0.01 0.01 0.005
- link RFsrFL_frame: mass None -> 2e-06; geometry collision box size=0.01 0.01 0.005
- link RFsrFR_frame: mass None -> 2e-06; geometry collision box size=0.01 0.01 0.005
- link RFsrRL_frame: mass None -> 2e-06; geometry collision box size=0.01 0.01 0.005
- link RFsrRR_frame: mass None -> 2e-06; geometry collision box size=0.01 0.01 0.005
Joints:
- removed joint CameraBottom_optical_frame_joint
- removed joint CameraTop_optical_frame_joint
- added joint CameraBottom_optical_frame_fixedjoint: type fixed, parent CameraBottom_frame, child CameraBottom_optical_frame, origin xyz=0 0 0 rpy=-1.57079632679 0 -1.57079632679
- added joint CameraTop_optical_frame_fixedjoint: type fixed, parent CameraTop_frame, child CameraTop_optical_frame, origin xyz=0 0 0 rpy=-1.57079632679 0 -1.57079632679

File: nao_description/urdf/naoV40_generated_urdf/nao_robot.xacro (robot description, xacro)
@@ -3,5 +3,5 @@
  ****** File automatically generated by generate_urdf.py script ******
  *********************************************************************-->
-<robot name="naoH25V40" xmlns:xacro="http://www.ros.org/wiki/xacro">
+<robot name="NaoH25V40" xmlns:xacro="http://www.ros.org/wiki/xacro">
 	<xacro:include filename="nao_visual_collisions.xacro"/>
 	<xacro:include filename="naoTransmission.xacro"/>

File: nao_description/urdf/naoV50_generated_urdf/nao.urdf (robot description, URDF)
Before this commit: robot naoH25V50, 79 links, 78 joints
Links:
- link LFsrFL_frame: mass None -> 2e-06; geometry collision box size=0.01 0.01 0.005
- link LFsrFR_frame: mass None -> 2e-06; geometry collision box size=0.01 0.01 0.005
- link LFsrRL_frame: mass None -> 2e-06; geometry collision box size=0.01 0.01 0.005
- link LFsrRR_frame: mass None -> 2e-06; geometry collision box size=0.01 0.01 0.005
- link RFsrFL_frame: mass None -> 2e-06; geometry collision box size=0.01 0.01 0.005
- link RFsrFR_frame: mass None -> 2e-06; geometry collision box size=0.01 0.01 0.005
- link RFsrRL_frame: mass None -> 2e-06; geometry collision box size=0.01 0.01 0.005
- link RFsrRR_frame: mass None -> 2e-06; geometry collision box size=0.01 0.01 0.005
Joints:
- removed joint CameraBottom_optical_frame_joint
- removed joint CameraTop_optical_frame_joint
- added joint CameraBottom_optical_frame_fixedjoint: type fixed, parent CameraBottom_frame, child CameraBottom_optical_frame, origin xyz=0 0 0 rpy=-1.57079632679 0 -1.57079632679
- added joint CameraTop_optical_frame_fixedjoint: type fixed, parent CameraTop_frame, child CameraTop_optical_frame, origin xyz=0 0 0 rpy=-1.57079632679 0 -1.57079632679

File: nao_description/urdf/naoV50_generated_urdf/nao_robot.xacro (robot description, xacro)
@@ -3,5 +3,5 @@
  ****** File automatically generated by generate_urdf.py script ******
  *********************************************************************-->
-<robot name="naoH25V50" xmlns:xacro="http://www.ros.org/wiki/xacro">
+<robot name="NaoH25V50" xmlns:xacro="http://www.ros.org/wiki/xacro">
 	<xacro:include filename="nao_visual_collisions.xacro"/>
 	<xacro:include filename="naoTransmission.xacro"/>

Commit message: update the .xacro / .urdf to the latest version of naoqi_tools

File: nao_description/urdf/naoV32_generated_urdf/nao.urdf (robot description, URDF)
Before this commit: robot naoH25V32, 77 links, 76 joints
Links:
- link LFsrFL_frame: mass None -> 2e-06; geometry collision box size=0.01 0.01 0.005
- link LFsrFR_frame: mass None -> 2e-06; geometry collision box size=0.01 0.01 0.005
- link LFsrRL_frame: mass None -> 2e-06; geometry collision box size=0.01 0.01 0.005
- link LFsrRR_frame: mass None -> 2e-06; geometry collision box size=0.01 0.01 0.005
- link RFsrFL_frame: mass None -> 2e-06; geometry collision box size=0.01 0.01 0.005
- link RFsrFR_frame: mass None -> 2e-06; geometry collision box size=0.01 0.01 0.005
- link RFsrRL_frame: mass None -> 2e-06; geometry collision box size=0.01 0.01 0.005
- link RFsrRR_frame: mass None -> 2e-06; geometry collision box size=0.01 0.01 0.005
Joints:
- removed joint CameraBottom_optical_frame_joint
- removed joint CameraTop_optical_frame_joint
- added joint CameraBottom_optical_frame_fixedjoint: type fixed, parent CameraBottom_frame, child CameraBottom_optical_frame, origin xyz=0 0 0 rpy=-1.57079632679 0 -1.57079632679
- added joint CameraTop_optical_frame_fixedjoint: type fixed, parent CameraTop_frame, child CameraTop_optical_frame, origin xyz=0 0 0 rpy=-1.57079632679 0 -1.57079632679

File: nao_description/urdf/naoV33_generated_urdf/nao.urdf (robot description, URDF)
Before this commit: robot naoH25V33, 83 links, 82 joints
Links:
- link LFsrFL_frame: mass None -> 2e-06; geometry collision box size=0.01 0.01 0.005
- link LFsrFR_frame: mass None -> 2e-06; geometry collision box size=0.01 0.01 0.005
- link LFsrRL_frame: mass None -> 2e-06; geometry collision box size=0.01 0.01 0.005
- link LFsrRR_frame: mass None -> 2e-06; geometry collision box size=0.01 0.01 0.005
- link RFsrFL_frame: mass None -> 2e-06; geometry collision box size=0.01 0.01 0.005
- link RFsrFR_frame: mass None -> 2e-06; geometry collision box size=0.01 0.01 0.005
- link RFsrRL_frame: mass None -> 2e-06; geometry collision box size=0.01 0.01 0.005
- link RFsrRR_frame: mass None -> 2e-06; geometry collision box size=0.01 0.01 0.005
Joints:
- removed joint CameraBottom_optical_frame_joint
- removed joint CameraTop_optical_frame_joint
- added joint CameraBottom_optical_frame_fixedjoint: type fixed, parent CameraBottom_frame, child CameraBottom_optical_frame, origin xyz=0 0 0 rpy=-1.57079632679 0 -1.57079632679
- added joint CameraTop_optical_frame_fixedjoint: type fixed, parent CameraTop_frame, child CameraTop_optical_frame, origin xyz=0 0 0 rpy=-1.57079632679 0 -1.57079632679

File: nao_description/urdf/naoV40_generated_urdf/nao.urdf (robot description, URDF)
Before this commit: robot naoH25V40, 83 links, 82 joints
Links:
- link LFsrFL_frame: mass None -> 2e-06; geometry collision box size=0.01 0.01 0.005
- link LFsrFR_frame: mass None -> 2e-06; geometry collision box size=0.01 0.01 0.005
- link LFsrRL_frame: mass None -> 2e-06; geometry collision box size=0.01 0.01 0.005
- link LFsrRR_frame: mass None -> 2e-06; geometry collision box size=0.01 0.01 0.005
- link RFsrFL_frame: mass None -> 2e-06; geometry collision box size=0.01 0.01 0.005
- link RFsrFR_frame: mass None -> 2e-06; geometry collision box size=0.01 0.01 0.005
- link RFsrRL_frame: mass None -> 2e-06; geometry collision box size=0.01 0.01 0.005
- link RFsrRR_frame: mass None -> 2e-06; geometry collision box size=0.01 0.01 0.005
Joints:
- removed joint CameraBottom_optical_frame_joint
- removed joint CameraTop_optical_frame_joint
- added joint CameraBottom_optical_frame_fixedjoint: type fixed, parent CameraBottom_frame, child CameraBottom_optical_frame, origin xyz=0 0 0 rpy=-1.57079632679 0 -1.57079632679
- added joint CameraTop_optical_frame_fixedjoint: type fixed, parent CameraTop_frame, child CameraTop_optical_frame, origin xyz=0 0 0 rpy=-1.57079632679 0 -1.57079632679

File: nao_description/urdf/naoV50_generated_urdf/nao.urdf (robot description, URDF)
Before this commit: robot naoH25V50, 79 links, 78 joints
Links:
- link LFsrFL_frame: mass None -> 2e-06; geometry collision box size=0.01 0.01 0.005
- link LFsrFR_frame: mass None -> 2e-06; geometry collision box size=0.01 0.01 0.005
- link LFsrRL_frame: mass None -> 2e-06; geometry collision box size=0.01 0.01 0.005
- link LFsrRR_frame: mass None -> 2e-06; geometry collision box size=0.01 0.01 0.005
- link RFsrFL_frame: mass None -> 2e-06; geometry collision box size=0.01 0.01 0.005
- link RFsrFR_frame: mass None -> 2e-06; geometry collision box size=0.01 0.01 0.005
- link RFsrRL_frame: mass None -> 2e-06; geometry collision box size=0.01 0.01 0.005
- link RFsrRR_frame: mass None -> 2e-06; geometry collision box size=0.01 0.01 0.005
Joints:
- removed joint CameraBottom_optical_frame_joint
- removed joint CameraTop_optical_frame_joint
- added joint CameraBottom_optical_frame_fixedjoint: type fixed, parent CameraBottom_frame, child CameraBottom_optical_frame, origin xyz=0 0 0 rpy=-1.57079632679 0 -1.57079632679
- added joint CameraTop_optical_frame_fixedjoint: type fixed, parent CameraTop_frame, child CameraTop_optical_frame, origin xyz=0 0 0 rpy=-1.57079632679 0 -1.57079632679
